Commit message: Fix joint order, joint resolution

File: ros2/src/k1_moveit/config/k1.ros2_control.xacro (robot description, xacro)
@@ -9,8 +9,22 @@
                 <param name="device">/dev/ttyAMA0</param>
             </hardware>
-            <joint name="right_hip">
+            <joint name="left_thigh">
                 <command_interface name="position"/>
                 <state_interface name="position">
-                  <param name="initial_value">${initial_positions['right_hip']}</param>
+                  <param name="initial_value">${initial_positions['left_thigh']}</param>
+                </state_interface>
+                <state_interface name="velocity"/>
+            </joint>
+            <joint name="left_knee">
+                <command_interface name="position"/>
+                <state_interface name="position">
+                  <param name="initial_value">${initial_positions['left_knee']}</param>
+                </state_interface>
+                <state_interface name="velocity"/>
+            </joint>
+            <joint name="left_calf">
+                <command_interface name="position"/>
+                <state_interface name="position">
+                  <param name="initial_value">${initial_positions['left_calf']}</param>
                 </state_interface>
                 <state_interface name="velocity"/>
@@ -37,8 +51,15 @@
                 <state_interface name="velocity"/>
             </joint>
-            <joint name="right_ankle">
+            <joint name="left_shoulder">
                 <command_interface name="position"/>
                 <state_interface name="position">
-                  <param name="initial_value">${initial_positions['right_ankle']}</param>
+                  <param name="initial_value">${initial_positions['left_shoulder']}</param>
+                </state_interface>
+                <state_interface name="velocity"/>
+            </joint>
+            <joint name="right_shoulder">
+                <command_interface name="position"/>
+                <state_interface name="position">
+                  <param name="initial_value">${initial_positions['right_shoulder']}</param>
                 </state_interface>
                 <state_interface name="velocity"/>
@@ -51,25 +72,4 @@
                 <state_interface name="velocity"/>
             </joint>
-            <joint name="left_thigh">
-                <command_interface name="position"/>
-                <state_interface name="position">
-                  <param name="initial_value">${initial_positions['left_thigh']}</param>
-                </state_interface>
-                <state_interface name="velocity"/>
-            </joint>
-            <joint name="left_knee">
-                <command_interface name="position"/>
-                <state_interface name="position">
-                  <param name="initial_value">${initial_positions['left_knee']}</param>
-                </state_interface>
-                <state_interface name="velocity"/>
-            </joint>
-            <joint name="left_calf">
-                <command_interface name="position"/>
-                <state_interface name="position">
-                  <param name="initial_value">${initial_positions['left_calf']}</param>
-                </state_interface>
-                <state_interface name="velocity"/>
-            </joint>
             <joint name="left_ankle">
                 <command_interface name="position"/>
@@ -79,8 +79,29 @@
                 <state_interface name="velocity"/>
             </joint>
-            <joint name="right_shoulder">
+            <joint name="right_hip">
                 <command_interface name="position"/>
                 <state_interface name="position">
-                  <param name="initial_value">${initial_positions['right_shoulder']}</param>
+                  <param name="initial_value">${initial_positions['right_hip']}</param>
+                </state_interface>
+                <state_interface name="velocity"/>
+            </joint>
+            <joint name="right_ankle">
+                <command_interface name="position"/>
+                <state_interface name="position">
+                  <param name="initial_value">${initial_positions['right_ankle']}</param>
+                </state_interface>
+                <state_interface name="velocity"/>
+            </joint>
+            <joint name="left_arm_upper">
+                <command_interface name="position"/>
+                <state_interface name="position">
+                  <param name="initial_value">${initial_positions['left_arm_upper']}</param>
+                </state_interface>
+                <state_interface name="velocity"/>
+            </joint>
+            <joint name="left_arm_lower">
+                <command_interface name="position"/>
+                <state_interface name="position">
+                  <param name="initial_value">${initial_positions['left_arm_lower']}</param>
                 </state_interface>
                 <state_interface name="velocity"/>
@@ -100,25 +121,4 @@
                 <state_interface name="velocity"/>
             </joint>
-            <joint name="left_shoulder">
-                <command_interface name="position"/>
-                <state_interface name="position">
-                  <param name="initial_value">${initial_positions['left_shoulder']}</param>
-                </state_interface>
-                <state_interface name="velocity"/>
-            </joint>
-            <joint name="left_arm_upper">
-                <command_interface name="position"/>
-                <state_interface name="position">
-                  <param name="initial_value">${initial_positions['left_arm_upper']}</param>
-                </state_interface>
-                <state_interface name="velocity"/>
-            </joint>
-            <joint name="left_arm_lower">
-                <command_interface name="position"/>
-                <state_interface name="position">
-                  <param name="initial_value">${initial_positions['left_arm_lower']}</param>
-                </state_interface>
-                <state_interface name="velocity"/>
-            </joint>
             <joint name="head">
                 <command_interface name="position"/>

Commit message: Fix order of joints to match hardware.
Signed-off-by: Curt Meyers <cmeyers@boilerbots.com>

File: ros2/src/k1_moveit/config/k1.ros2_control.xacro (robot description, xacro)
@@ -12,8 +12,22 @@
                 <param name="device">/dev/ttyAMA0</param>
             </hardware>
-            <joint name="right_hip_joint">
+            <joint name="left_thigh_joint">
                 <command_interface name="position"/>
                 <state_interface name="position">
-                  <param name="initial_value">${initial_positions['right_hip_joint']}</param>
+                  <param name="initial_value">${initial_positions['left_thigh_joint']}</param>
+                </state_interface>
+                <state_interface name="velocity"/>
+            </joint>
+            <joint name="left_knee_joint">
+                <command_interface name="position"/>
+                <state_interface name="position">
+                  <param name="initial_value">${initial_positions['left_knee_joint']}</param>
+                </state_interface>
+                <state_interface name="velocity"/>
+            </joint>
+            <joint name="left_calf_joint">
+                <command_interface name="position"/>
+                <state_interface name="position">
+                  <param name="initial_value">${initial_positions['left_calf_joint']}</param>
                 </state_interface>
                 <state_interface name="velocity"/>
@@ -40,8 +54,15 @@
                 <state_interface name="velocity"/>
             </joint>
-            <joint name="right_ankle_joint">
+            <joint name="left_shoulder_joint">
                 <command_interface name="position"/>
                 <state_interface name="position">
-                  <param name="initial_value">${initial_positions['right_ankle_joint']}</param>
+                  <param name="initial_value">${initial_positions['left_shoulder_joint']}</param>
+                </state_interface>
+                <state_interface name="velocity"/>
+            </joint>
+            <joint name="right_shoulder_joint">
+                <command_interface name="position"/>
+                <state_interface name="position">
+                  <param name="initial_value">${initial_positions['right_shoulder_joint']}</param>
                 </state_interface>
                 <state_interface name="velocity"/>
@@ -54,25 +75,4 @@
                 <state_interface name="velocity"/>
             </joint>
-            <joint name="left_thigh_joint">
-                <command_interface name="position"/>
-                <state_interface name="position">
-                  <param name="initial_value">${initial_positions['left_thigh_joint']}</param>
-                </state_interface>
-                <state_interface name="velocity"/>
-            </joint>
-            <joint name="left_knee_joint">
-                <command_interface name="position"/>
-                <state_interface name="position">
-                  <param name="initial_value">${initial_positions['left_knee_joint']}</param>
-                </state_interface>
-                <state_interface name="velocity"/>
-            </joint>
-            <joint name="left_calf_joint">
-                <command_interface name="position"/>
-                <state_interface name="position">
-                  <param name="initial_value">${initial_positions['left_calf_joint']}</param>
-                </state_interface>
-                <state_interface name="velocity"/>
-            </joint>
             <joint name="left_ankle_joint">
                 <command_interface name="position"/>
@@ -82,8 +82,29 @@
                 <state_interface name="velocity"/>
             </joint>
-            <joint name="right_shoulder_joint">
+            <joint name="right_hip_joint">
                 <command_interface name="position"/>
                 <state_interface name="position">
-                  <param name="initial_value">${initial_positions['right_shoulder_joint']}</param>
+                  <param name="initial_value">${initial_positions['right_hip_joint']}</param>
+                </state_interface>
+                <state_interface name="velocity"/>
+            </joint>
+            <joint name="right_ankle_joint">
+                <command_interface name="position"/>
+                <state_interface name="position">
+                  <param name="initial_value">${initial_positions['right_ankle_joint']}</param>
+                </state_interface>
+                <state_interface name="velocity"/>
+            </joint>
+            <joint name="left_upper_arm_joint">
+                <command_interface name="position"/>
+                <state_interface name="position">
+                  <param name="initial_value">${initial_positions['left_upper_arm_joint']}</param>
+                </state_interface>
+                <state_interface name="velocity"/>
+            </joint>
+            <joint name="left_lower_arm_joint">
+                <command_interface name="position"/>
+                <state_interface name="position">
+                  <param name="initial_value">${initial_positions['left_lower_arm_joint']}</param>
                 </state_interface>
                 <state_interface name="velocity"/>
@@ -103,25 +124,4 @@
                 <state_interface name="velocity"/>
             </joint>
-            <joint name="left_shoulder_joint">
-                <command_interface name="position"/>
-                <state_interface name="position">
-                  <param name="initial_value">${initial_positions['left_shoulder_joint']}</param>
-                </state_interface>
-                <state_interface name="velocity"/>
-            </joint>
-            <joint name="left_upper_arm_joint">
-                <command_interface name="position"/>
-                <state_interface name="position">
-                  <param name="initial_value">${initial_positions['left_upper_arm_joint']}</param>
-                </state_interface>
-                <state_interface name="velocity"/>
-            </joint>
-            <joint name="left_lower_arm_joint">
-                <command_interface name="position"/>
-                <state_interface name="position">
-                  <param name="initial_value">${initial_positions['left_lower_arm_joint']}</param>
-                </state_interface>
-                <state_interface name="velocity"/>
-            </joint>
             <joint name="head_joint">
                 <command_interface name="position"/>
