Commit message: Adding moveit configuration
The planner doesn't work, something wrong with the velocity limits or some other
bug in the current rolling implementation.

Signed-off-by: Curt Meyers <cmeyers@boilerbots.com>

File: ros2/src/k1_description/urdf/k1.xacro (robot description, xacro)
@@ -49,5 +49,5 @@
     <child link="right_hip_link" />
     <axis xyz="0 1 0" />
-    <limit lower="-1.5" upper="1.5" effort="0" velocity="0" />
+    <limit lower="-1.5" upper="1.5" effort="0" velocity="3" />
   </joint>
   <link name="right_thigh_link">
@@ -78,5 +78,5 @@
     <child link="right_thigh_link" />
     <axis xyz="0 1 0" />
-    <limit lower="-3" upper="3" effort="0" velocity="0" />
+    <limit lower="-3" upper="3" effort="0" velocity="3" />
   </joint>
   <link name="right_knee_link">
@@ -107,5 +107,5 @@
     <child link="right_knee_link" />
     <axis xyz="0 1 0" />
-    <limit lower="-3" upper="3" effort="0" velocity="0" />
+    <limit lower="-3" upper="3" effort="0" velocity="3" />
   </joint>
   <link name="right_calf_link">
@@ -136,5 +136,5 @@
     <child link="right_calf_link" />
     <axis xyz="0 1 0" />
-    <limit lower="-3" upper="3" effort="0" velocity="0" />
+    <limit lower="-3" upper="3" effort="0" velocity="3" />
   </joint>
   <link name="right_ankle_link">
@@ -165,5 +165,5 @@
     <child link="right_ankle_link" />
     <axis xyz="0 1 0" />
-    <limit lower="-3" upper="3" effort="0" velocity="0" />
+    <limit lower="-3" upper="3" effort="0" velocity="3" />
   </joint>
   <link name="left_hip_link">
@@ -194,5 +194,5 @@
     <child link="left_hip_link" />
     <axis xyz="0 1 0" />
-    <limit lower="-3" upper="3" effort="0" velocity="0" />
+    <limit lower="-3" upper="3" effort="0" velocity="3" />
   </joint>
   <link name="left_thigh_link">
@@ -223,5 +223,5 @@
     <child link="left_thigh_link" />
     <axis xyz="0 1 0" />
-    <limit lower="-3" upper="3" effort="0" velocity="0" />
+    <limit lower="-3" upper="3" effort="0" velocity="3" />
   </joint>
   <link name="left_knee_link">
@@ -252,5 +252,5 @@
     <child link="left_knee_link" />
     <axis xyz="0 1 0" />
-    <limit lower="-3" upper="3" effort="0" velocity="0" />
+    <limit lower="-3" upper="3" effort="0" velocity="3" />
   </joint>
   <link name="left_calf_link">
@@ -281,5 +281,5 @@
     <child link="left_calf_link" />
     <axis xyz="0 1 0" />
-    <limit lower="-3" upper="3" effort="0" velocity="0" />
+    <limit lower="-3" upper="3" effort="0" velocity="3" />
   </joint>
   <link name="left_ankle_link">
@@ -310,5 +310,5 @@
     <child link="left_ankle_link" />
     <axis xyz="0 1 0" />
-    <limit lower="-3" upper="3" effort="0" velocity="0" />
+    <limit lower="-3" upper="3" effort="0" velocity="3" />
   </joint>
   <link name="right_arm_link">
@@ -339,5 +339,5 @@
     <child link="right_arm_link" />
     <axis xyz="0 1 0" />
-    <limit lower="-3" upper="3" effort="0" velocity="0" />
+    <limit lower="-3" upper="3" effort="0" velocity="3" />
   </joint>
   <link name="right_arm_upper">
@@ -368,5 +368,5 @@
     <child link="right_arm_upper" />
     <axis xyz="0 1 0" />
-    <limit lower="-3" upper="3" effort="0" velocity="0" />
+    <limit lower="-3" upper="3" effort="0" velocity="3" />
   </joint>
   <link name="right_arm_lower">
@@ -397,5 +397,5 @@
     <child link="right_arm_lower" />
     <axis xyz="0 1 0" />
-    <limit lower="-3" upper="3" effort="0" velocity="0" />
+    <limit lower="-3" upper="3" effort="0" velocity="3" />
   </joint>
   <link name="left_arm_link">
@@ -426,5 +426,5 @@
     <child link="left_arm_link" />
     <axis xyz="0 1 0" />
-    <limit lower="-3" upper="3" effort="0" velocity="0" />
+    <limit lower="-3" upper="3" effort="0" velocity="3" />
   </joint>
   <link name="left_arm_upper_link">
@@ -455,5 +455,5 @@
     <child link="left_arm_upper_link" />
     <axis xyz="0 1 0" />
-    <limit lower="-3" upper="3" effort="0" velocity="0" />
+    <limit lower="-3" upper="3" effort="0" velocity="3" />
   </joint>
   <link name="left_arm_lower_link">
@@ -484,5 +484,5 @@
     <child link="left_arm_lower_link" />
     <axis xyz="0 1 0" />
-    <limit lower="-3" upper="3" effort="0" velocity="0" />
+    <limit lower="-3" upper="3" effort="0" velocity="3" />
   </joint>
   <link name="head_link">
@@ -513,5 +513,5 @@
     <child link="head_link" />
     <axis xyz="0 -1 0" />
-    <limit lower="-3" upper="3" effort="0" velocity="0" />
+    <limit lower="-3" upper="3" effort="0" velocity="3" />
   </joint>
 </robot>

Commit message: Fix MoveIt configuration problems
There are problems with Rolling configurations that need to be manually fixed.

Signed-off-by: Curt Meyers <cmeyers@boilerbots.com>

File: ros2/src/k1_description/urdf/k1.xacro (robot description, xacro)
@@ -49,5 +49,5 @@
     <child link="right_hip_link" />
     <axis xyz="0 1 0" />
-    <limit lower="-1.5" upper="1.5" effort="0" velocity="3" />
+    <limit lower="-1.5" upper="1.5" effort="0" velocity="3.0" />
   </joint>
   <link name="right_thigh_link">
@@ -78,5 +78,5 @@
     <child link="right_thigh_link" />
     <axis xyz="0 1 0" />
-    <limit lower="-3" upper="3" effort="0" velocity="3" />
+    <limit lower="-3" upper="3" effort="0" velocity="3.0" />
   </joint>
   <link name="right_knee_link">
@@ -107,5 +107,5 @@
     <child link="right_knee_link" />
     <axis xyz="0 1 0" />
-    <limit lower="-3" upper="3" effort="0" velocity="3" />
+    <limit lower="-3" upper="3" effort="0" velocity="3.0" />
   </joint>
   <link name="right_calf_link">
@@ -136,5 +136,5 @@
     <child link="right_calf_link" />
     <axis xyz="0 1 0" />
-    <limit lower="-3" upper="3" effort="0" velocity="3" />
+    <limit lower="-3" upper="3" effort="0" velocity="3.0" />
   </joint>
   <link name="right_ankle_link">
@@ -165,5 +165,5 @@
     <child link="right_ankle_link" />
     <axis xyz="0 1 0" />
-    <limit lower="-3" upper="3" effort="0" velocity="3" />
+    <limit lower="-3" upper="3" effort="0" velocity="3.0" />
   </joint>
   <link name="left_hip_link">
@@ -194,5 +194,5 @@
     <child link="left_hip_link" />
     <axis xyz="0 1 0" />
-    <limit lower="-3" upper="3" effort="0" velocity="3" />
+    <limit lower="-3" upper="3" effort="0" velocity="3.0" />
   </joint>
   <link name="left_thigh_link">
@@ -223,5 +223,5 @@
     <child link="left_thigh_link" />
     <axis xyz="0 1 0" />
-    <limit lower="-3" upper="3" effort="0" velocity="3" />
+    <limit lower="-3" upper="3" effort="0" velocity="3.0" />
   </joint>
   <link name="left_knee_link">
@@ -252,5 +252,5 @@
     <child link="left_knee_link" />
     <axis xyz="0 1 0" />
-    <limit lower="-3" upper="3" effort="0" velocity="3" />
+    <limit lower="-3" upper="3" effort="0" velocity="3.0" />
   </joint>
   <link name="left_calf_link">
@@ -281,5 +281,5 @@
     <child link="left_calf_link" />
     <axis xyz="0 1 0" />
-    <limit lower="-3" upper="3" effort="0" velocity="3" />
+    <limit lower="-3" upper="3" effort="0" velocity="3.0" />
   </joint>
   <link name="left_ankle_link">
@@ -310,5 +310,5 @@
     <child link="left_ankle_link" />
     <axis xyz="0 1 0" />
-    <limit lower="-3" upper="3" effort="0" velocity="3" />
+    <limit lower="-3" upper="3" effort="0" velocity="3.0" />
   </joint>
   <link name="right_arm_link">
@@ -339,5 +339,5 @@
     <child link="right_arm_link" />
     <axis xyz="0 1 0" />
-    <limit lower="-3" upper="3" effort="0" velocity="3" />
+    <limit lower="-3" upper="3" effort="0" velocity="3.0" />
   </joint>
   <link name="right_arm_upper">
@@ -368,5 +368,5 @@
     <child link="right_arm_upper" />
     <axis xyz="0 1 0" />
-    <limit lower="-3" upper="3" effort="0" velocity="3" />
+    <limit lower="-3" upper="3" effort="0" velocity="3.0" />
   </joint>
   <link name="right_arm_lower">
@@ -397,5 +397,5 @@
     <child link="right_arm_lower" />
     <axis xyz="0 1 0" />
-    <limit lower="-3" upper="3" effort="0" velocity="3" />
+    <limit lower="-3" upper="3" effort="0" velocity="3.0" />
   </joint>
   <link name="left_arm_link">
@@ -426,5 +426,5 @@
     <child link="left_arm_link" />
     <axis xyz="0 1 0" />
-    <limit lower="-3" upper="3" effort="0" velocity="3" />
+    <limit lower="-3" upper="3" effort="0" velocity="3.0" />
   </joint>
   <link name="left_arm_upper_link">
@@ -455,5 +455,5 @@
     <child link="left_arm_upper_link" />
     <axis xyz="0 1 0" />
-    <limit lower="-3" upper="3" effort="0" velocity="3" />
+    <limit lower="-3" upper="3" effort="0" velocity="3.0" />
   </joint>
   <link name="left_arm_lower_link">
@@ -484,5 +484,5 @@
     <child link="left_arm_lower_link" />
     <axis xyz="0 1 0" />
-    <limit lower="-3" upper="3" effort="0" velocity="3" />
+    <limit lower="-3" upper="3" effort="0" velocity="3.0" />
   </joint>
   <link name="head_link">
@@ -513,5 +513,5 @@
     <child link="head_link" />
     <axis xyz="0 -1 0" />
-    <limit lower="-3" upper="3" effort="0" velocity="3" />
+    <limit lower="-3" upper="3" effort="0" velocity="3.0" />
   </joint>
 </robot>
