Commit message: Updated k1_description again
Fixed joints and links and an axis problem on the arm_lower.

Signed-off-by: Curt Meyers <cmeyers@boilerbots.com>

File: ros2/src/k1_description/urdf/k1.xacro (robot description, xacro)
@@ -2,7 +2,7 @@
   <link name="base_link">
     <inertial>
-      <origin xyz="-2.74854541183482E-18 -4.61950778389125E-19 0.0470916230366492" rpy="0 0 0" />
-      <mass value="0.2292" />
-      <inertia ixx="0.00022678767591623" ixy="-3.7704942585474E-21" ixz="-1.16227512873892E-21" iyy="0.00015895767591623" iyz="-2.76736603223311E-21" izz="0.00012895" />
+      <origin xyz="3.1237E-05 -2.6609E-18 0.043467" rpy="0 0 0" />
+      <mass value="0.24447" />
+      <inertia ixx="0.00022866" ixy="-4.4957E-21" ixz="-1.1924E-22" iyy="0.00016383" iyz="-2.1079E-21" izz="0.00013299" />
     </inertial>
     <visual>
@@ -12,5 +12,5 @@
       </geometry>
       <material name="">
-        <color rgba="0.792156862745098 0.819607843137255 0.933333333333333 1" />
+        <color rgba="0.79216 0.81961 0.93333 1" />
       </material>
     </visual>
@@ -24,7 +24,7 @@
   <link name="right_hip_link">
     <inertial>
-      <origin xyz="-0.00651824599613865 2.92734586571086E-18 -0.00228432235654178" rpy="0 0 0" />
-      <mass value="0.027821769923242" />
-      <inertia ixx="4.43354161733857E-06" ixy="4.67010169351549E-23" ixz="4.767222976598E-08" iyy="3.78674573990841E-06" iyz="-5.11832663195711E-22" izz="5.52212734276756E-06" />
+      <origin xyz="-0.0091911 0.00013724 0.0068616" rpy="0 0 0" />
+      <mass value="0.027822" />
+      <inertia ixx="2.9324E-06" ixy="5.4126E-22" ixz="8.2036E-08" iyy="5.289E-06" iyz="-5.5232E-22" izz="5.521E-06" />
     </inertial>
     <visual>
@@ -34,5 +34,5 @@
       </geometry>
       <material name="">
-        <color rgba="0.250980392156863 0.250980392156863 0.250980392156863 1" />
+        <color rgba="0.25098 0.25098 0.25098 1" />
       </material>
     </visual>
@@ -44,16 +44,16 @@
     </collision>
   </link>
-  <joint name="right_hip" type="revolute">
+  <joint name="right_hip" type="continuous">
     <origin xyz="0.0005 -0.015 -0.02" rpy="-3.1416 0 1.5708" />
     <parent link="base_link" />
     <child link="right_hip_link" />
     <axis xyz="0 1 0" />
-    <limit lower="-1.5" upper="1.5" effort="0" velocity="3.0" />
+    <limit lower="0" upper="0" effort="0" velocity="0" />
   </joint>
   <link name="right_thigh_link">
     <inertial>
-      <origin xyz="6.31352746712905E-05 -1.04083408558608E-17 0.00403162866350376" rpy="0 0 0" />
-      <mass value="0.0278217699232421" />
-      <inertia ixx="5.93907846618009E-06" ixy="-2.07567490117999E-22" ixz="1.05342441330196E-08" iyy="3.78674573990841E-06" iyz="4.94440913447292E-22" izz="4.01659049392605E-06" />
+      <origin xyz="0.00048354 -1.0408E-17 0.028801" rpy="0 0 0" />
+      <mass value="0.044066" />
+      <inertia ixx="6.9987E-06" ixy="2.4849E-23" ixz="6.6075E-07" iyy="5.8317E-06" iyz="-2.5887E-22" izz="4.6055E-06" />
     </inertial>
     <visual>
@@ -63,5 +63,5 @@
       </geometry>
       <material name="">
-        <color rgba="0.250980392156863 0.250980392156863 0.250980392156863 1" />
+        <color rgba="0.25098 0.25098 0.25098 1" />
       </material>
     </visual>
@@ -73,16 +73,16 @@
     </collision>
   </link>
-  <joint name="right_thigh" type="revolute">
+  <joint name="right_thigh" type="continuous">
     <origin xyz="-0.0094505 0.0005 0.033316" rpy="0.031659 0.025339 1.5716" />
     <parent link="right_hip_link" />
     <child link="right_thigh_link" />
     <axis xyz="0 1 0" />
-    <limit lower="-3" upper="3" effort="0" velocity="3.0" />
+    <limit lower="0" upper="0" effort="0" velocity="0" />
   </joint>
   <link name="right_knee_link">
     <inertial>
-      <origin xyz="-0.000135799465695009 1.04083408558608E-17 -0.00634963453755198" rpy="0 0 0" />
-      <mass value="0.0315177699232421" />
-      <inertia ixx="6.03248087268701E-06" ixy="-5.67084596461784E-22" ixz="2.17227530672295E-07" iyy="3.91569507324175E-06" iyz="2.21803588059263E-22" izz="4.53508142075247E-06" />
+      <origin xyz="-0.0178121084477415 2.77555756156289E-17 0.0307655812522569" rpy="0 0 0" />
+      <mass value="0.032371769923242" />
+      <inertia ixx="6.0588731794123E-06" ixy="-3.9527863778785E-22" ixz="3.4680753923887E-07" iyy="3.93488969546397E-06" iyz="4.3890533855335E-22" izz="4.63947306958273E-06" />
     </inertial>
     <visual>
@@ -92,5 +92,5 @@
       </geometry>
       <material name="">
-        <color rgba="0.250980392156863 0.250980392156863 0.250980392156863 1" />
+        <color rgba="0.752941176470588 1 1 1" />
       </material>
     </visual>
@@ -102,16 +102,16 @@
     </collision>
   </link>
-  <joint name="right_knee" type="revolute">
+  <joint name="right_knee" type="continuous">
     <origin xyz="-0.0021501 0 0.055492" rpy="0 0.49935 -3.1416" />
     <parent link="right_thigh_link" />
     <child link="right_knee_link" />
     <axis xyz="0 1 0" />
-    <limit lower="-3" upper="3" effort="0" velocity="3.0" />
+    <limit lower="0" upper="0" effort="0" velocity="0" />
   </joint>
   <link name="right_calf_link">
     <inertial>
-      <origin xyz="-0.000387072019440708 0 0.0083418498895714" rpy="0 0 0" />
-      <mass value="0.032371769923242" />
-      <inertia ixx="6.27933649382619E-06" ixy="1.2046713659036E-21" ixz="-1.02631006855728E-07" iyy="3.93488969546397E-06" iyz="3.11525357236097E-22" izz="4.41900975516884E-06" />
+      <origin xyz="-0.009582 0.0010801 -0.024645" rpy="0 0 0" />
+      <mass value="0.027822" />
+      <inertia ixx="5.3156E-06" ixy="1.0464E-21" ixz="7.4393E-08" iyy="2.9298E-06" iyz="-2.516E-22" izz="5.497E-06" />
     </inertial>
     <visual>
@@ -121,5 +121,5 @@
       </geometry>
       <material name="">
-        <color rgba="0.792156862745098 0.819607843137255 0.933333333333333 1" />
+        <color rgba="0.75294 1 1 1" />
       </material>
     </visual>
@@ -131,16 +131,16 @@
     </collision>
   </link>
-  <joint name="right_calf" type="revolute">
+  <joint name="right_calf" type="continuous">
     <origin xyz="-0.023084 0 0.051939" rpy="3.1416 -0.11317 0" />
     <parent link="right_knee_link" />
     <child link="right_calf_link" />
     <axis xyz="0 1 0" />
-    <limit lower="-3" upper="3" effort="0" velocity="3.0" />
+    <limit lower="0" upper="0" effort="0" velocity="0" />
   </joint>
   <link name="right_ankle_link">
     <inertial>
-      <origin xyz="-0.012895367887895 0.00398487631475268 0.0116977656940815" rpy="0 0 0" />
-      <mass value="0.152373296152955" />
-      <inertia ixx="0.000107106171742906" ixy="-2.67854466622824E-10" ixz="4.02982212640107E-07" iyy="4.5135980483168E-05" iyz="1.35813174315468E-10" izz="0.000140258354090534" />
+      <origin xyz="-0.0134919017266966 0.00459336693369054 0.0134840145322273" rpy="0 0 0" />
+      <mass value="0.132188163411726" />
+      <inertia ixx="0.000105111740356927" ixy="-2.67854466622719E-10" ixz="4.02982212640105E-07" iyy="4.22846170003843E-05" iyz="1.35813174315627E-10" izz="0.000136756609487253" />
     </inertial>
     <visual>
@@ -150,5 +150,5 @@
       </geometry>
       <material name="">
-        <color rgba="0.250980392156863 0.250980392156863 0.250980392156863 1" />
+        <color rgba="0.752941176470588 1 1 1" />
       </material>
     </visual>
@@ -160,16 +160,16 @@
     </collision>
   </link>
-  <joint name="right_ankle" type="revolute">
+  <joint name="right_ankle" type="continuous">
     <origin xyz="-0.012051 -0.0075 -0.030737" rpy="2.7982 0 -1.5708" />
     <parent link="right_calf_link" />
     <child link="right_ankle_link" />
     <axis xyz="0 1 0" />
-    <limit lower="-3" upper="3" effort="0" velocity="3.0" />
+    <limit lower="0" upper="0" effort="0" velocity="0" />
   </joint>
   <link name="left_hip_link">
     <inertial>
-      <origin xyz="-0.00245265378337689 1.30104260698261E-18 -0.00695509378336099" rpy="0 0 0" />
+      <origin xyz="0.00574384356514769 0.000137242116570632 -0.00899186986767261" rpy="0 0 0" />
       <mass value="0.027821769923242" />
-      <inertia ixx="5.53623440177927E-06" ixy="-6.75016664722994E-22" ixz="-7.12623027855017E-08" iyy="3.78674573990841E-06" iyz="1.56369646485007E-22" izz="4.41943455832686E-06" />
+      <inertia ixx="5.52363659732332E-06" ixy="2.35404777695923E-22" ixz="9.52912065661088E-22" iyy="5.28896445958682E-06" iyz="-7.01815773253074E-22" izz="2.92981364310441E-06" />
     </inertial>
     <visual>
@@ -189,16 +189,16 @@
     </collision>
   </link>
-  <joint name="left_hip" type="revolute">
+  <joint name="left_hip" type="continuous">
     <origin xyz="0.0005 0.015 -0.02" rpy="3.1416 1.3958 1.5708" />
     <parent link="base_link" />
     <child link="left_hip_link" />
     <axis xyz="0 1 0" />
-    <limit lower="-3" upper="3" effort="0" velocity="3.0" />
+    <limit lower="0" upper="0" effort="0" velocity="0" />
   </joint>
   <link name="left_thigh_link">
     <inertial>
-      <origin xyz="-0.000293046937027548 6.93889390390723E-18 -0.00404812796646236" rpy="0 0 0" />
-      <mass value="0.0278217699232421" />
-      <inertia ixx="5.93359082667115E-06" ixy="1.4430802527091E-22" ixz="4.85714473787366E-08" iyy="3.78674573990841E-06" iyz="1.27893144976878E-21" izz="4.02207813343499E-06" />
+      <origin xyz="0.000483541080447515 -1.38777878078145E-17 -0.0288011243914165" rpy="0 0 0" />
+      <mass value="0.0440662654824574" />
+      <inertia ixx="6.99871657924005E-06" ixy="-1.30252055807653E-21" ixz="-6.60751594534272E-07" iyy="5.83167629890069E-06" iyz="1.22954384106141E-21" izz="4.6055287326144E-06" />
     </inertial>
     <visual>
@@ -218,16 +218,16 @@
     </collision>
   </link>
-  <joint name="left_thigh" type="revolute">
-    <origin xyz="0.03 0.000500000000000008 -0.00899999999999999" rpy="-1.5707963267949 0 1.4528659227743" />
+  <joint name="left_thigh" type="continuous">
+    <origin xyz="0.03 0.0005 -0.009" rpy="-1.5708 0 1.4529" />
     <parent link="left_hip_link" />
     <child link="left_thigh_link" />
     <axis xyz="0 1 0" />
-    <limit lower="-3" upper="3" effort="0" velocity="3.0" />
+    <limit lower="0" upper="0" effort="0" velocity="0" />
   </joint>
   <link name="left_knee_link">
     <inertial>
-      <origin xyz="-4.89852228429261E-05 -1.76941794549634E-16 0.00624714520731363" rpy="0 0 0" />
-      <mass value="0.031517769923242" />
-      <inertia ixx="6.0575195240443E-06" ixy="-4.30509763183972E-22" ixz="-2.21402757576364E-07" iyy="3.91569507324175E-06" iyz="-6.18830948968168E-22" izz="4.51004276939517E-06" />
+      <origin xyz="-0.0159002354975483 -6.76542155630955E-16 -0.0317958284727074" rpy="0 0 0" />
+      <mass value="0.0323717699232421" />
+      <inertia ixx="6.09585578173946E-06" ixy="-9.75086376578192E-22" ixz="-2.57710392869743E-07" iyy="3.93488969546397E-06" iyz="-1.37120055400643E-21" izz="4.60249046725557E-06" />
     </inertial>
     <visual>
@@ -237,5 +237,5 @@
       </geometry>
       <material name="">
-        <color rgba="0.250980392156863 0.250980392156863 0.250980392156863 1" />
+        <color rgba="0.752941176470588 1 1 1" />
       </material>
     </visual>
@@ -247,16 +247,16 @@
     </collision>
   </link>
-  <joint name="left_knee" type="revolute">
-    <origin xyz="-0.00215005179923169 0 -0.0554917017754941" rpy="0 -0.499346721680133 3.14159265358979" />
+  <joint name="left_knee" type="continuous">
+    <origin xyz="-0.0021501 0 -0.055492" rpy="0 -0.49935 3.1416" />
     <parent link="left_thigh_link" />
     <child link="left_knee_link" />
     <axis xyz="0 1 0" />
-    <limit lower="-3" upper="3" effort="0" velocity="3.0" />
+    <limit lower="0" upper="0" effort="0" velocity="0" />
   </joint>
   <link name="left_calf_link">
     <inertial>
-      <origin xyz="-0.000168198425069349 -1.45716771982052E-16 -0.00827653769580036" rpy="0 0 0" />
-      <mass value="0.0323717699232421" />
-      <inertia ixx="6.3036101539097E-06" ixy="2.11807547460393E-22" ixz="6.55798264311812E-08" iyy="3.93488969546398E-06" iyz="-1.59430620853435E-21" izz="4.39473609508533E-06" />
+      <origin xyz="-0.00690141207525505 0.00108014351796133 0.0255261573931621" rpy="0 0 0" />
+      <mass value="0.0278217699232421" />
+      <inertia ixx="5.30185932211653E-06" ixy="3.09254745805148E-23" ixz="-5.34769808048693E-08" iyy="2.92981364310441E-06" iyz="-8.94604079450337E-22" izz="5.51074173479362E-06" />
     </inertial>
     <visual>
@@ -266,5 +266,5 @@
       </geometry>
       <material name="">
-        <color rgba="0.250980392156863 0.250980392156863 0.250980392156863 1" />
+        <color rgba="0.752941176470588 1 1 1" />
       </material>
     </visual>
@@ -276,16 +276,16 @@
     </collision>
   </link>
-  <joint name="left_calf" type="revolute">
-    <origin xyz="-0.0198692740011601 0 -0.0532513355105156" rpy="-3.14159265358979 0.0520650640700285 0" />
+  <joint name="left_calf" type="continuous">
+    <origin xyz="-0.019869 0 -0.053251" rpy="-3.1416 0.052065 0" />
     <parent link="left_knee_link" />
     <child link="left_calf_link" />
     <axis xyz="0 1 0" />
-    <limit lower="-3" upper="3" effort="0" velocity="3.0" />
+    <limit lower="0" upper="0" effort="0" velocity="0" />
   </joint>
   <link name="left_ankle_link">
     <inertial>
-      <origin xyz="-0.0118168931644879 -0.00398488608298372 -0.0127751448550284" rpy="0 0 0" />
-      <mass value="0.152373247707281" />
-      <inertia ixx="0.000140255620895985" ixy="-5.26733657775849E-10" ixz="-7.25991197394405E-07" iyy="4.51378245971644E-05" iyz="-7.24960113436985E-11" izz="0.000107122876890634" />
+      <origin xyz="-0.0136213334288442 -0.00459337841653701 -0.013353320848436" rpy="0 0 0" />
+      <mass value="0.132188114966052" />
+      <inertia ixx="0.000136753876292704" ixy="-5.26733657769073E-10" ixz="-7.25991197394409E-07" iyy="4.22864611143807E-05" iyz="-7.24960113429766E-11" izz="0.000105128445504655" />
     </inertial>
     <visual>
@@ -295,5 +295,5 @@
       </geometry>
       <material name="">
-        <color rgba="0.250980392156863 0.250980392156863 0.250980392156863 1" />
+        <color rgba="0.752941176470588 1 1 1" />
       </material>
     </visual>
@@ -305,16 +305,16 @@
     </collision>
   </link>
-  <joint name="left_ankle" type="revolute">
-    <origin xyz="-0.00870769361648834 -0.0074999999999989 0.0318461311917393" rpy="1.57079632679489 1.33418390311996 0" />
+  <joint name="left_ankle" type="continuous">
+    <origin xyz="-0.0087077 -0.0075 0.031846" rpy="1.5708 1.3342 0" />
     <parent link="left_calf_link" />
     <child link="left_ankle_link" />
     <axis xyz="0 1 0" />
-    <limit lower="-3" upper="3" effort="0" velocity="3.0" />
+    <limit lower="0" upper="0" effort="0" velocity="0" />
   </joint>
   <link name="right_arm_link">
     <inertial>
-      <origin xyz="6.93889390390723E-17 -0.00711626473085393 -0.00652151176940128" rpy="0 0 0" />
-      <mass value="0.027821769923242" />
-      <inertia ixx="5.93916106248708E-06" ixy="-3.23486617911071E-22" ixz="-1.66478749847302E-08" iyy="4.87325547682611E-06" iyz="-5.55023094980973E-22" izz="2.92999816070136E-06" />
+      <origin xyz="-9.99200722162641E-16 0.0259259508257144 -2.15105711021124E-16" rpy="0 0 0" />
+      <mass value="0.00763663718201332" />
+      <inertia ixx="2.43758966616897E-06" ixy="2.93020214434485E-22" ixz="4.12200417999712E-09" iyy="2.02189199404243E-06" iyz="5.46092272261234E-23" izz="9.35393567758914E-07" />
     </inertial>
     <visual>
@@ -324,5 +324,5 @@
       </geometry>
       <material name="">
-        <color rgba="0.250980392156863 0.250980392156863 0.250980392156863 1" />
+        <color rgba="0.752941176470588 1 1 1" />
       </material>
     </visual>
@@ -334,21 +334,21 @@
     </collision>
   </link>
-  <joint name="right_shoulder" type="revolute">
-    <origin xyz="-0.007 -0.026 0.075" rpy="0 -1.5708 0" />
+  <joint name="right_shoulder" type="continuous">
+    <origin xyz="-0.007 -0.026 0.075" rpy="3.1416 -1.5708 0" />
     <parent link="base_link" />
     <child link="right_arm_link" />
     <axis xyz="0 1 0" />
-    <limit lower="-3" upper="3" effort="0" velocity="3.0" />
-  </joint>
-  <link name="right_arm_upper">
-    <inertial>
-      <origin xyz="-2.56739074444567E-16 -4.77048955893622E-16 -0.027997650371616" rpy="0 0 0" />
+    <limit lower="0" upper="0" effort="0" velocity="0" />
+  </joint>
+  <link name="right_arm_upper_link">
+    <inertial>
+      <origin xyz="-0.0267099408480544 -5.91540705308091E-16 -0.00839330007950644" rpy="0 0 0" />
       <mass value="0.0404127433991118" />
-      <inertia ixx="5.83338324794275E-06" ixy="9.26442286059391E-23" ixz="6.64109709606441E-22" iyy="6.27306084712394E-06" iyz="-4.91345283856498E-22" izz="5.2865719936405E-06" />
-    </inertial>
-    <visual>
-      <origin xyz="0 0 0" rpy="0 0 0" />
-      <geometry>
-        <mesh filename="package://k1_description/meshes/visual/right_arm_upper.STL" />
+      <inertia ixx="5.33571477961189E-06" ixy="-3.15155813382704E-22" ixz="-1.56386748236192E-07" iyy="6.27306084712395E-06" iyz="-1.94387443949962E-22" izz="5.78424046197137E-06" />
+    </inertial>
+    <visual>
+      <origin xyz="0 0 0" rpy="0 0 0" />
+      <geometry>
+        <mesh filename="package://k1_description/meshes/visual/right_arm_upper_link.STL" />
       </geometry>
       <material name="">
@@ -359,25 +359,25 @@
       <origin xyz="0 0 0" rpy="0 0 0" />
       <geometry>
-        <mesh filename="package://k1_description/meshes/collision/right_arm_upper.STL" />
-      </geometry>
-    </collision>
-  </link>
-  <joint name="right_upper" type="revolute">
-    <origin xyz="0 -0.0350000000000004 0" rpy="-1.56717278184304 0.010474038342865 0.333073638779225" />
+        <mesh filename="package://k1_description/meshes/collision/right_arm_upper_link.STL" />
+      </geometry>
+    </collision>
+  </link>
+  <joint name="right_upper" type="continuous">
+    <origin xyz="0 0.0350000000000004 0" rpy="-1.56989921107132 -0.00259316215202615 -0.33306656840474" />
     <parent link="right_arm_link" />
-    <child link="right_arm_upper" />
-    <axis xyz="0 1 0" />
-    <limit lower="-3" upper="3" effort="0" velocity="3.0" />
-  </joint>
-  <link name="right_arm_lower">
-    <inertial>
-      <origin xyz="3.33066907387547E-16 0.000840716498841119 -0.018261633701405" rpy="0 0 0" />
+    <child link="right_arm_upper_link" />
+    <axis xyz="0 1 0" />
+    <limit lower="0" upper="0" effort="0" velocity="0" />
+  </joint>
+  <link name="right_arm_lower_link">
+    <inertial>
+      <origin xyz="0.0182616337014053 0.00084071649884114 -4.33680868994202E-18" rpy="0 0 0" />
       <mass value="0.0290848600660391" />
-      <inertia ixx="4.64311633086366E-06" ixy="3.30872245021211E-23" ixz="-1.58818677610181E-21" iyy="4.0538898836655E-06" iyz="1.67669592897643E-07" izz="2.72498939319332E-06" />
-    </inertial>
-    <visual>
-      <origin xyz="0 0 0" rpy="0 0 0" />
-      <geometry>
-        <mesh filename="package://k1_description/meshes/visual/right_arm_lower.STL" />
+      <inertia ixx="2.72498939319332E-06" ixy="-1.67669592897643E-07" ixz="2.5146290621612E-22" iyy="4.0538898836655E-06" iyz="3.57083530681485E-22" izz="4.64311633086366E-06" />
+    </inertial>
+    <visual>
+      <origin xyz="0 0 0" rpy="0 0 0" />
+      <geometry>
+        <mesh filename="package://k1_description/meshes/visual/right_arm_lower_link.STL" />
       </geometry>
       <material name="">
@@ -388,20 +388,20 @@
       <origin xyz="0 0 0" rpy="0 0 0" />
       <geometry>
-        <mesh filename="package://k1_description/meshes/collision/right_arm_lower.STL" />
-      </geometry>
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