Commit message: Inching closer to a working moveit configuration
Signed-off-by: Curt Meyers <cmeyers@boilerbots.com>

File: ros2/src/k1_description/urdf/k1.xacro (robot description, xacro)
@@ -44,10 +44,10 @@
     </collision>
   </link>
-  <joint name="right_hip" type="continuous">
+  <joint name="right_hip" type="revolute">
     <origin xyz="0.0005 -0.015 -0.02" rpy="-3.1416 0 1.5708" />
     <parent link="base_link" />
     <child link="right_hip_link" />
     <axis xyz="0 1 0" />
-    <limit lower="0" upper="0" effort="0" velocity="0" />
+    <limit lower="-3.0" upper="3.0" effort="1000" velocity="3.0" />
   </joint>
   <link name="right_thigh_link">
@@ -73,10 +73,10 @@
     </collision>
   </link>
-  <joint name="right_thigh" type="continuous">
+  <joint name="right_thigh" type="revolute">
     <origin xyz="-0.0094505 0.0005 0.033316" rpy="0.031659 0.025339 1.5716" />
     <parent link="right_hip_link" />
     <child link="right_thigh_link" />
     <axis xyz="0 1 0" />
-    <limit lower="0" upper="0" effort="0" velocity="0" />
+    <limit lower="-3.0" upper="3.0" effort="1000" velocity="3.0" />
   </joint>
   <link name="right_knee_link">
@@ -102,10 +102,10 @@
     </collision>
   </link>
-  <joint name="right_knee" type="continuous">
+  <joint name="right_knee" type="revolute">
     <origin xyz="-0.0021501 0 0.055492" rpy="0 0.49935 -3.1416" />
     <parent link="right_thigh_link" />
     <child link="right_knee_link" />
     <axis xyz="0 1 0" />
-    <limit lower="0" upper="0" effort="0" velocity="0" />
+    <limit lower="-3.0" upper="3.0" effort="1000" velocity="3.0" />
   </joint>
   <link name="right_calf_link">
@@ -131,10 +131,10 @@
     </collision>
   </link>
-  <joint name="right_calf" type="continuous">
+  <joint name="right_calf" type="revolute">
     <origin xyz="-0.023084 0 0.051939" rpy="3.1416 -0.11317 0" />
     <parent link="right_knee_link" />
     <child link="right_calf_link" />
     <axis xyz="0 1 0" />
-    <limit lower="0" upper="0" effort="0" velocity="0" />
+    <limit lower="-3.0" upper="3.0" effort="1000" velocity="3.0" />
   </joint>
   <link name="right_ankle_link">
@@ -160,10 +160,10 @@
     </collision>
   </link>
-  <joint name="right_ankle" type="continuous">
+  <joint name="right_ankle" type="revolute">
     <origin xyz="-0.012051 -0.0075 -0.030737" rpy="2.7982 0 -1.5708" />
     <parent link="right_calf_link" />
     <child link="right_ankle_link" />
     <axis xyz="0 1 0" />
-    <limit lower="0" upper="0" effort="0" velocity="0" />
+    <limit lower="-3.0" upper="3.0" effort="1000" velocity="3.0" />
   </joint>
   <link name="left_hip_link">
@@ -189,10 +189,10 @@
     </collision>
   </link>
-  <joint name="left_hip" type="continuous">
+  <joint name="left_hip" type="revolute">
     <origin xyz="0.0005 0.015 -0.02" rpy="3.1416 1.3958 1.5708" />
     <parent link="base_link" />
     <child link="left_hip_link" />
     <axis xyz="0 1 0" />
-    <limit lower="0" upper="0" effort="0" velocity="0" />
+    <limit lower="-3.0" upper="3.0" effort="1000" velocity="3.0" />
   </joint>
   <link name="left_thigh_link">
@@ -218,10 +218,10 @@
     </collision>
   </link>
-  <joint name="left_thigh" type="continuous">
+  <joint name="left_thigh" type="revolute">
     <origin xyz="0.03 0.0005 -0.009" rpy="-1.5708 0 1.4529" />
     <parent link="left_hip_link" />
     <child link="left_thigh_link" />
     <axis xyz="0 1 0" />
-    <limit lower="0" upper="0" effort="0" velocity="0" />
+    <limit lower="-3.0" upper="3.0" effort="1000" velocity="3.0" />
   </joint>
   <link name="left_knee_link">
@@ -247,10 +247,10 @@
     </collision>
   </link>
-  <joint name="left_knee" type="continuous">
+  <joint name="left_knee" type="revolute">
     <origin xyz="-0.0021501 0 -0.055492" rpy="0 -0.49935 3.1416" />
     <parent link="left_thigh_link" />
     <child link="left_knee_link" />
     <axis xyz="0 1 0" />
-    <limit lower="0" upper="0" effort="0" velocity="0" />
+    <limit lower="-3.0" upper="3.0" effort="1000" velocity="3.0" />
   </joint>
   <link name="left_calf_link">
@@ -276,10 +276,10 @@
     </collision>
   </link>
-  <joint name="left_calf" type="continuous">
+  <joint name="left_calf" type="revolute">
     <origin xyz="-0.019869 0 -0.053251" rpy="-3.1416 0.052065 0" />
     <parent link="left_knee_link" />
     <child link="left_calf_link" />
     <axis xyz="0 1 0" />
-    <limit lower="0" upper="0" effort="0" velocity="0" />
+    <limit lower="-3.0" upper="3.0" effort="1000" velocity="3.0" />
   </joint>
   <link name="left_ankle_link">
@@ -305,10 +305,10 @@
     </collision>
   </link>
-  <joint name="left_ankle" type="continuous">
+  <joint name="left_ankle" type="revolute">
     <origin xyz="-0.0087077 -0.0075 0.031846" rpy="1.5708 1.3342 0" />
     <parent link="left_calf_link" />
     <child link="left_ankle_link" />
     <axis xyz="0 1 0" />
-    <limit lower="0" upper="0" effort="0" velocity="0" />
+    <limit lower="-3.0" upper="3.0" effort="1000" velocity="3.0" />
   </joint>
   <link name="right_arm_link">
@@ -334,10 +334,10 @@
     </collision>
   </link>
-  <joint name="right_shoulder" type="continuous">
+  <joint name="right_shoulder" type="revolute">
     <origin xyz="-0.007 -0.026 0.075" rpy="3.1416 -1.5708 0" />
     <parent link="base_link" />
     <child link="right_arm_link" />
     <axis xyz="0 1 0" />
-    <limit lower="0" upper="0" effort="0" velocity="0" />
+    <limit lower="-3.0" upper="3.0" effort="1000" velocity="3.0" />
   </joint>
   <link name="right_arm_upper_link">
@@ -363,10 +363,10 @@
     </collision>
   </link>
-  <joint name="right_upper" type="continuous">
+  <joint name="right_upper" type="revolute">
     <origin xyz="0 0.0350000000000004 0" rpy="-1.56989921107132 -0.00259316215202615 -0.33306656840474" />
     <parent link="right_arm_link" />
     <child link="right_arm_upper_link" />
     <axis xyz="0 1 0" />
-    <limit lower="0" upper="0" effort="0" velocity="0" />
+    <limit lower="-3.0" upper="3.0" effort="1000" velocity="3.0" />
   </joint>
   <link name="right_arm_lower_link">
@@ -392,10 +392,10 @@
     </collision>
   </link>
-  <joint name="right_arm_lower" type="continuous">
+  <joint name="right_arm_lower" type="revolute">
     <origin xyz="-0.0667804560220959 0 -0.0209850111622641" rpy="1.5864967516128 0.304075688258208 -3.0891987069566" />
     <parent link="right_arm_upper_link" />
     <child link="right_arm_lower_link" />
     <axis xyz="0 1 0" />
-    <limit lower="0" upper="0" effort="0" velocity="0" />
+    <limit lower="-3.0" upper="3.0" effort="1000" velocity="3.0" />
   </joint>
   <link name="left_arm_link">
@@ -421,10 +421,10 @@
     </collision>
   </link>
-  <joint name="left_shoulder" type="continuous">
+  <joint name="left_shoulder" type="revolute">
     <origin xyz="-0.007 0.026 0.075" rpy="3.1416 -1.5708 0" />
     <parent link="base_link" />
     <child link="left_arm_link" />
     <axis xyz="0 1 0" />
-    <limit lower="0" upper="0" effort="0" velocity="0" />
+    <limit lower="-3.0" upper="3.0" effort="1000" velocity="3.0" />
   </joint>
   <link name="left_arm_upper_link">
@@ -450,10 +450,10 @@
     </collision>
   </link>
-  <joint name="left_arm_upper" type="continuous">
+  <joint name="left_arm_upper" type="revolute">
     <origin xyz="0 -0.0350000000000004 0" rpy="1.57169344251847 0.00259316215202667 0.33306656840474" />
     <parent link="left_arm_link" />
     <child link="left_arm_upper_link" />
     <axis xyz="0 1 0" />
-    <limit lower="0" upper="0" effort="0" velocity="0" />
+    <limit lower="-3.0" upper="3.0" effort="1000" velocity="3.0" />
   </joint>
   <link name="left_arm_lower_link">
@@ -479,10 +479,10 @@
     </collision>
   </link>
-  <joint name="left_arm_lower" type="continuous">
+  <joint name="left_arm_lower" type="revolute">
     <origin xyz="-0.0667804560220957 0 -0.020985011162264" rpy="1.5864967516128 0.304075688258208 -3.0891987069566" />
     <parent link="left_arm_upper_link" />
     <child link="left_arm_lower_link" />
     <axis xyz="0 1 0" />
-    <limit lower="0" upper="0" effort="0" velocity="0" />
+    <limit lower="-3.0" upper="3.0" effort="1000" velocity="3.0" />
   </joint>
   <link name="head_link">
@@ -513,5 +513,5 @@
     <child link="head_link" />
     <axis xyz="0 1 0" />
-    <limit lower="0" upper="0" effort="0" velocity="0" />
+    <limit lower="-3.0" upper="3.0" effort="1000" velocity="3.0" />
   </joint>
 </robot>

Commit message: Update k1_description
Adding fixed joints for hands and feet.

Signed-off-by: Curt Meyers <cmeyers@boilerbots.com>

File: ros2/src/k1_description/urdf/k1.xacro (robot description, xacro)
@@ -312,4 +312,32 @@
     <limit lower="-3.0" upper="3.0" effort="1000" velocity="3.0" />
   </joint>
+  <link name="left_foot_link">
+    <inertial>
+      <origin xyz="1.35029760289784E-08 0.0104287918497478 1.17152012257815E-08" rpy="0 0 0" />
+      <mass value="0.124551473427286" />
+      <inertia ixx="4.13510775251367E-05" ixy="5.14922415404396E-10" ixz="8.73800926913661E-11" iyy="0.000134748648682341" iyz="1.37529274140502E-10" izz="0.000102674182175629" />
+    </inertial>
+    <visual>
+      <origin xyz="0 0 0" rpy="0 0 0" />
+      <geometry>
+        <mesh filename="package://k1_description/meshes/visual/left_foot_link.STL" />
+      </geometry>
+      <material name="">
+        <color rgba="1 1 0.752941176470588 1" />
+      </material>
+    </visual>
+    <collision>
+      <origin xyz="0 0 0" rpy="0 0 0" />
+      <geometry>
+        <mesh filename="package://k1_description/meshes/collision/left_foot_link.STL" />
+      </geometry>
+    </collision>
+  </link>
+  <joint name="left_foot_joint" type="fixed">
+    <origin xyz="-0.0254952367690822 0.0113755745672261 0.00285705310295755" rpy="-0.0314669727072048 0 -1.5707963267949" />
+    <parent link="left_ankle_link" />
+    <child link="left_foot_link" />
+    <axis xyz="0 0 0" />
+  </joint>
   <link name="right_arm_link">
     <inertial>
@@ -399,4 +427,60 @@
     <limit lower="-3.0" upper="3.0" effort="1000" velocity="3.0" />
   </joint>
+  <link name="right_hand_link">
+    <inertial>
+      <origin xyz="-0.00274751358458329 -2.60208521396521E-18 0.0122930084282204" rpy="0 0 0" />
+      <mass value="0.00889972732481042" />
+      <inertia ixx="1.20252640088182E-06" ixy="-2.36586579887237E-23" ixz="1.67669592897643E-07" iyy="1.14137172758277E-06" iyz="1.91905902112302E-22" izz="7.3055800721365E-07" />
+    </inertial>
+    <visual>
+      <origin xyz="0 0 0" rpy="0 0 0" />
+      <geometry>
+        <mesh filename="package://k1_description/meshes/visual/right_hand_link.STL" />
+      </geometry>
+      <material name="">
+        <color rgba="1 1 1 1" />
+      </material>
+    </visual>
+    <collision>
+      <origin xyz="0 0 0" rpy="0 0 0" />
+      <geometry>
+        <mesh filename="package://k1_description/meshes/collision/right_hand_link.STL" />
+      </geometry>
+    </collision>
+  </link>
+  <joint name="right_hand_joint" type="fixed">
+    <origin xyz="0.0269999999999999 0 0" rpy="-1.5707963267949 0 -1.5707963267949" />
+    <parent link="right_arm_lower_link" />
+    <child link="right_hand_link" />
+    <axis xyz="0 0 0" />
+  </joint>
+  <link name="right_foot_link">
+    <inertial>
+      <origin xyz="3.89163107121504E-10 0.0104288935743586 5.67569245074617E-09" rpy="0 0 0" />
+      <mass value="0.124551526229713" />
+      <inertia ixx="4.13492347432596E-05" ixy="-1.32395086473111E-10" ixz="2.69560335696787E-10" iyy="0.000134739848442081" iyz="3.6269551537831E-10" izz="0.000102669008431253" />
+    </inertial>
+    <visual>
+      <origin xyz="0 0 0" rpy="0 0 0" />
+      <geometry>
+        <mesh filename="package://k1_description/meshes/visual/right_foot_link.STL" />
+      </geometry>
+      <material name="">
+        <color rgba="1 1 0.752941176470588 1" />
+      </material>
+    </visual>
+    <collision>
+      <origin xyz="0 0 0" rpy="0 0 0" />
+      <geometry>
+        <mesh filename="package://k1_description/meshes/collision/right_foot_link.STL" />
+      </geometry>
+    </collision>
+  </link>
+  <joint name="right_foot_joint" type="fixed">
+    <origin xyz="0.0437300656421878 -0.00156463412465353 0.200047116627725" rpy="-1.49777528191655 -0.0646765133830734 1.56982137043522" />
+    <parent link="right_hand_link" />
+    <child link="right_foot_link" />
+    <axis xyz="0 0 0" />
+  </joint>
   <link name="left_arm_link">
     <inertial>
@@ -486,4 +570,32 @@
     <limit lower="-3.0" upper="3.0" effort="1000" velocity="3.0" />
   </joint>
+  <link name="left_hand_link">
+    <inertial>
+      <origin xyz="-0.00274751358458326 0 0.0122930084282204" rpy="0 0 0" />
+      <mass value="0.00889972732481043" />
+      <inertia ixx="1.20252640088182E-06" ixy="4.72850042347696E-23" ixz="1.67669592897643E-07" iyy="1.14137172758278E-06" iyz="-5.9557004103818E-23" izz="7.30558007213651E-07" />
+    </inertial>
+    <visual>
+      <origin xyz="0 0 0" rpy="0 0 0" />
+      <geometry>
+        <mesh filename="package://k1_description/meshes/visual/left_hand_link.STL" />
+      </geometry>
+      <material name="">
+        <color rgba="1 1 1 1" />
+      </material>
+    </visual>
+    <collision>
+      <origin xyz="0 0 0" rpy="0 0 0" />
+      <geometry>
+        <mesh filename="package://k1_description/meshes/collision/left_hand_link.STL" />
+      </geometry>
+    </collision>
+  </link>
+  <joint name="left_hand_joint" type="fixed">
+    <origin xyz="0.0269999999999999 0 0" rpy="-1.5707963267949 0 -1.57079632679489" />
+    <parent link="left_arm_lower_link" />
+    <child link="left_hand_link" />
+    <axis xyz="0 0 0" />
+  </joint>
   <link name="head_link">
     <inertial>

Commit message: Fix hand link
Signed-off-by: Curt Meyers <cmeyers@boilerbots.com>

File: ros2/src/k1_description/urdf/k1.xacro (robot description, xacro)
@@ -166,4 +166,32 @@
     <axis xyz="0 1 0" />
     <limit lower="-3.0" upper="3.0" effort="1000" velocity="3.0" />
+  </joint>
+  <link name="right_foot_link">
+    <inertial>
+      <origin xyz="3.89163107121504E-10 0.0104288935743586 5.67569245074617E-09" rpy="0 0 0" />
+      <mass value="0.124551526229713" />
+      <inertia ixx="4.13492347432596E-05" ixy="-1.32395086473482E-10" ixz="2.69560335696801E-10" iyy="0.000134739848442081" iyz="3.62695515377463E-10" izz="0.000102669008431253" />
+    </inertial>
+    <visual>
+      <origin xyz="0 0 0" rpy="0 0 0" />
+      <geometry>
+        <mesh filename="package://k1_description/meshes/visual/right_foot_link.STL" />
+      </geometry>
+      <material name="">
+        <color rgba="1 1 0.752941176470588 1" />
+      </material>
+    </visual>
+    <collision>
+      <origin xyz="0 0 0" rpy="0 0 0" />
+      <geometry>
+        <mesh filename="package://k1_description/meshes/collision/right_foot_link.STL" />
+      </geometry>
+    </collision>
+  </link>
+  <joint name="right_foot_joint" type="fixed">
+    <origin xyz="-0.014194 0.004875 0.024182" rpy="-1.5581 0 1.5708" />
+    <parent link="right_ankle_link" />
+    <child link="right_foot_link" />
+    <axis xyz="0 0 0" />
   </joint>
   <link name="left_hip_link">
@@ -427,60 +455,4 @@
     <limit lower="-3.0" upper="3.0" effort="1000" velocity="3.0" />
   </joint>
-  <link name="right_hand_link">
-    <inertial>
-      <origin xyz="-0.00274751358458329 -2.60208521396521E-18 0.0122930084282204" rpy="0 0 0" />
-      <mass value="0.00889972732481042" />
-      <inertia ixx="1.20252640088182E-06" ixy="-2.36586579887237E-23" ixz="1.67669592897643E-07" iyy="1.14137172758277E-06" iyz="1.91905902112302E-22" izz="7.3055800721365E-07" />
-    </inertial>
-    <visual>
-      <origin xyz="0 0 0" rpy="0 0 0" />
-      <geometry>
-        <mesh filename="package://k1_description/meshes/visual/right_hand_link.STL" />
-      </geometry>
-      <material name="">
-        <color rgba="1 1 1 1" />
-      </material>
-    </visual>
-    <collision>
-      <origin xyz="0 0 0" rpy="0 0 0" />
-      <geometry>
-        <mesh filename="package://k1_description/meshes/collision/right_hand_link.STL" />
-      </geometry>
-    </collision>
-  </link>
-  <joint name="right_hand_joint" type="fixed">
-    <origin xyz="0.0269999999999999 0 0" rpy="-1.5707963267949 0 -1.5707963267949" />
-    <parent link="right_arm_lower_link" />
-    <child link="right_hand_link" />
-    <axis xyz="0 0 0" />
-  </joint>
-  <link name="right_foot_link">
-    <inertial>
-      <origin xyz="3.89163107121504E-10 0.0104288935743586 5.67569245074617E-09" rpy="0 0 0" />
-      <mass value="0.124551526229713" />
-      <inertia ixx="4.13492347432596E-05" ixy="-1.32395086473111E-10" ixz="2.69560335696787E-10" iyy="0.000134739848442081" iyz="3.6269551537831E-10" izz="0.000102669008431253" />
-    </inertial>
-    <visual>
-      <origin xyz="0 0 0" rpy="0 0 0" />
-      <geometry>
-        <mesh filename="package://k1_description/meshes/visual/right_foot_link.STL" />
-      </geometry>
-      <material name="">
-        <color rgba="1 1 0.752941176470588 1" />
-      </material>
-    </visual>
-    <collision>
-      <origin xyz="0 0 0" rpy="0 0 0" />
-      <geometry>
-        <mesh filename="package://k1_description/meshes/collision/right_foot_link.STL" />
-      </geometry>
-    </collision>
-  </link>
-  <joint name="right_foot_joint" type="fixed">
-    <origin xyz="0.0437300656421878 -0.00156463412465353 0.200047116627725" rpy="-1.49777528191655 -0.0646765133830734 1.56982137043522" />
-    <parent link="right_hand_link" />
-    <child link="right_foot_link" />
-    <axis xyz="0 0 0" />
-  </joint>
   <link name="left_arm_link">
     <inertial>
@@ -627,3 +599,31 @@
     <limit lower="-3.0" upper="3.0" effort="1000" velocity="3.0" />
   </joint>
+  <link name="face_link">
+    <inertial>
+      <origin xyz="-5.27015314794538E-07 0.0192636340735728 -1.77662602571516E-05" rpy="0 0 0" />
+      <mass value="0.0901518210219852" />
+      <inertia ixx="3.42226307311124E-05" ixy="4.62380615190735E-10" ixz="1.35489424526232E-09" iyy="3.57923710083382E-05" iyz="-6.15798115932383E-09" izz="2.41005619280376E-05" />
+    </inertial>
+    <visual>
+      <origin xyz="0 0 0" rpy="0 0 0" />
+      <geometry>
+        <mesh filename="package://k1_description/meshes/visual/face_link.STL" />
+      </geometry>
+      <material name="">
+        <color rgba="1 0.501960784313725 1 1" />
+      </material>
+    </visual>
+    <collision>
+      <origin xyz="0 0 0" rpy="0 0 0" />
+      <geometry>
+        <mesh filename="package://k1_description/meshes/collision/face_link.STL" />
+      </geometry>
+    </collision>
+  </link>
+  <joint name="face_joint" type="fixed">
+    <origin xyz="0 0 0" rpy="3.1416 0 0" />
+    <parent link="head_link" />
+    <child link="face_link" />
+    <axis xyz="0 0 0" />
+  </joint>
 </robot>

Commit message: Still fixing description, right hand was missing
Signed-off-by: Curt Meyers <cmeyers@boilerbots.com>

File: ros2/src/k1_description/urdf/k1.xacro (robot description, xacro)
@@ -455,4 +455,32 @@
     <limit lower="-3.0" upper="3.0" effort="1000" velocity="3.0" />
   </joint>
+  <link name="right_hand_link">
+    <inertial>
+      <origin xyz="-0.00274751358458329 -2.60208521396521E-18 0.0122930084282204" rpy="0 0 0" />
+      <mass value="0.00889972732481042" />
+      <inertia ixx="1.20252640088182E-06" ixy="-2.53130192138298E-23" ixz="1.67669592897643E-07" iyy="1.14137172758277E-06" iyz="1.91905902112302E-22" izz="7.3055800721365E-07" />
+    </inertial>
+    <visual>
+      <origin xyz="0 0 0" rpy="0 0 0" />
+      <geometry>
+        <mesh filename="package://k1_description/meshes/visual/right_hand_link.STL" />
+      </geometry>
+      <material name="">
+        <color rgba="1 1 1 1" />
+      </material>
+    </visual>
+    <collision>
+      <origin xyz="0 0 0" rpy="0 0 0" />
+      <geometry>
+        <mesh filename="package://k1_description/meshes/collision/right_hand_link.STL" />
+      </geometry>
+    </collision>
+  </link>
+  <joint name="right_hand_joint" type="fixed">
+    <origin xyz="0.0269999999999999 0 0" rpy="-1.5707963267949 0 -1.5707963267949" />
+    <parent link="right_arm_lower_link" />
+    <child link="right_hand_link" />
+    <axis xyz="0 0 0" />
+  </joint>
   <link name="left_arm_link">
     <inertial>
