Commit message: more xacro changes Signed-off-by: Curt Meyers <cmeyers@boilerbots.com>

File: ros2/src/k1_description/urdf/k1.xacro (robot description, xacro)
@@ -1,8 +1,8 @@
-<robot name="k1">
+<robot name="k1_with_hands">
   <link name="base_link">
     <inertial>
-      <origin xyz="3.1237E-05 -2.6609E-18 0.043467" rpy="0 0 0" />
-      <mass value="0.24447" />
-      <inertia ixx="0.00022866" ixy="-4.4957E-21" ixz="-1.1924E-22" iyy="0.00016383" iyz="-2.1079E-21" izz="0.00013299" />
+      <origin xyz="-2.7485E-18 -4.6195E-19 0.047092" rpy="0 0 0" />
+      <mass value="0.2292" />
+      <inertia ixx="0.00022679" ixy="-3.7705E-21" ixz="-1.2088E-21" iyy="0.00015896" iyz="-2.7674E-21" izz="0.00012895" />
     </inertial>
     <visual>
@@ -24,7 +24,7 @@
   <link name="right_hip_link">
     <inertial>
-      <origin xyz="-0.0091911 0.00013724 0.0068616" rpy="0 0 0" />
-      <mass value="0.027822" />
-      <inertia ixx="2.9324E-06" ixy="5.4126E-22" ixz="8.2036E-08" iyy="5.289E-06" iyz="-5.5232E-22" izz="5.521E-06" />
+      <origin xyz="-0.0091910773470667 0.000137242116570623 0.00686156682154296" rpy="0 0 0" />
+      <mass value="0.027821769923242" />
+      <inertia ixx="2.93241080676327E-06" ixy="5.41152994005165E-22" ixz="8.20355865167775E-08" iyy="5.28896445958682E-06" iyz="-5.59192783257843E-22" izz="5.52103943366446E-06" />
     </inertial>
     <visual>
@@ -34,5 +34,5 @@
       </geometry>
       <material name="">
-        <color rgba="0.25098 0.25098 0.25098 1" />
+        <color rgba="0.250980392156863 0.250980392156863 0.250980392156863 1" />
       </material>
     </visual>
@@ -49,11 +49,11 @@
     <child link="right_hip_link" />
     <axis xyz="0 1 0" />
-    <limit lower="-3.0" upper="3.0" effort="1000" velocity="3.0" />
+    <limit lower="-6.28" upper="6.28" effort="1.0" velocity="3.0" />
   </joint>
   <link name="right_thigh_link">
     <inertial>
-      <origin xyz="0.00048354 -1.0408E-17 0.028801" rpy="0 0 0" />
-      <mass value="0.044066" />
-      <inertia ixx="6.9987E-06" ixy="2.4849E-23" ixz="6.6075E-07" iyy="5.8317E-06" iyz="-2.5887E-22" izz="4.6055E-06" />
+      <origin xyz="0.000483541080447617 -1.04083408558608E-17 0.0288011243914165" rpy="0 0 0" />
+      <mass value="0.0440662654824575" />
+      <inertia ixx="6.99871657924006E-06" ixy="2.48488152353851E-23" ixz="6.60751594534264E-07" iyy="5.83167629890069E-06" iyz="-2.58865577893623E-22" izz="4.6055287326144E-06" />
     </inertial>
     <visual>
@@ -63,5 +63,5 @@
       </geometry>
       <material name="">
-        <color rgba="0.25098 0.25098 0.25098 1" />
+        <color rgba="0.250980392156863 0.250980392156863 0.250980392156863 1" />
       </material>
     </visual>
@@ -74,15 +74,15 @@
   </link>
   <joint name="right_thigh" type="revolute">
-    <origin xyz="-0.0094505 0.0005 0.033316" rpy="0.031659 0.025339 1.5716" />
+    <origin xyz="-0.00945051849090369 0.000499999999999996 0.0333157275209935" rpy="0.0316585832535403 0.0253385921253171 1.57159869279353" />
     <parent link="right_hip_link" />
     <child link="right_thigh_link" />
     <axis xyz="0 1 0" />
-    <limit lower="-3.0" upper="3.0" effort="1000" velocity="3.0" />
+    <limit lower="-6.28" upper="6.28" effort="1.0" velocity="1.0" />
   </joint>
   <link name="right_knee_link">
     <inertial>
-      <origin xyz="-0.0178121084477415 2.77555756156289E-17 0.0307655812522569" rpy="0 0 0" />
+      <origin xyz="-0.0178121084477415 3.81639164714898E-17 0.0307655812522569" rpy="0 0 0" />
       <mass value="0.032371769923242" />
-      <inertia ixx="6.0588731794123E-06" ixy="-3.9527863778785E-22" ixz="3.4680753923887E-07" iyy="3.93488969546397E-06" iyz="4.3890533855335E-22" izz="4.63947306958273E-06" />
+      <inertia ixx="6.0588731794123E-06" ixy="-3.78363821203638E-22" ixz="3.46807539238869E-07" iyy="3.93488969546397E-06" iyz="4.20940815551816E-22" izz="4.63947306958273E-06" />
     </inertial>
     <visual>
@@ -103,15 +103,15 @@
   </link>
   <joint name="right_knee" type="revolute">
-    <origin xyz="-0.0021501 0 0.055492" rpy="0 0.49935 -3.1416" />
+    <origin xyz="-0.00215005179923145 0 0.0554917017754941" rpy="0 0.499346721680126 -3.14159265358979" />
     <parent link="right_thigh_link" />
     <child link="right_knee_link" />
     <axis xyz="0 1 0" />
-    <limit lower="-3.0" upper="3.0" effort="1000" velocity="3.0" />
+    <limit lower="-6.28" upper="6.28" effort="1.0" velocity="1.0" />
   </joint>
   <link name="right_calf_link">
     <inertial>
-      <origin xyz="-0.009582 0.0010801 -0.024645" rpy="0 0 0" />
-      <mass value="0.027822" />
-      <inertia ixx="5.3156E-06" ixy="1.0464E-21" ixz="7.4393E-08" iyy="2.9298E-06" iyz="-2.516E-22" izz="5.497E-06" />
+      <origin xyz="-0.00958197752831114 0.00108014351796196 -0.0246454845060883" rpy="0 0 0" />
+      <mass value="0.0278217699232421" />
+      <inertia ixx="5.31556206114482E-06" ixy="1.0431771588901E-21" ixz="7.43927658286799E-08" iyy="2.92981364310441E-06" iyz="-2.7149420750487E-22" izz="5.49703899576533E-06" />
     </inertial>
     <visual>
@@ -121,5 +121,5 @@
       </geometry>
       <material name="">
-        <color rgba="0.75294 1 1 1" />
+        <color rgba="0.752941176470588 1 1 1" />
       </material>
     </visual>
@@ -132,9 +132,9 @@
   </link>
   <joint name="right_calf" type="revolute">
-    <origin xyz="-0.023084 0 0.051939" rpy="3.1416 -0.11317 0" />
+    <origin xyz="-0.0230838749026589 0 0.0519386898416303" rpy="3.14159265358979 -0.113165928627979 0" />
     <parent link="right_knee_link" />
     <child link="right_calf_link" />
     <axis xyz="0 1 0" />
-    <limit lower="-3.0" upper="3.0" effort="1000" velocity="3.0" />
+    <limit lower="-6.28" upper="6.28" effort="1.0" velocity="1.0" />
   </joint>
   <link name="right_ankle_link">
@@ -142,5 +142,5 @@
       <origin xyz="-0.0134919017266966 0.00459336693369054 0.0134840145322273" rpy="0 0 0" />
       <mass value="0.132188163411726" />
-      <inertia ixx="0.000105111740356927" ixy="-2.67854466622719E-10" ixz="4.02982212640105E-07" iyy="4.22846170003843E-05" iyz="1.35813174315627E-10" izz="0.000136756609487253" />
+      <inertia ixx="0.000105111740356927" ixy="-2.67854466622726E-10" ixz="4.02982212640105E-07" iyy="4.22846170003843E-05" iyz="1.35813174315733E-10" izz="0.000136756609487253" />
     </inertial>
     <visual>
@@ -161,9 +161,9 @@
   </link>
   <joint name="right_ankle" type="revolute">
-    <origin xyz="-0.012051 -0.0075 -0.030737" rpy="2.7982 0 -1.5708" />
+    <origin xyz="-0.0120513798099409 -0.00749999999999831 -0.0307370174980681" rpy="2.79822593138815 0 -1.5707963267949" />
     <parent link="right_calf_link" />
     <child link="right_ankle_link" />
     <axis xyz="0 1 0" />
-    <limit lower="-3.0" upper="3.0" effort="1000" velocity="3.0" />
+    <limit lower="-6.28" upper="6.28" effort="1.0" velocity="1.0" />
   </joint>
   <link name="right_foot_link">
@@ -171,5 +171,5 @@
       <origin xyz="3.89163107121504E-10 0.0104288935743586 5.67569245074617E-09" rpy="0 0 0" />
       <mass value="0.124551526229713" />
-      <inertia ixx="4.13492347432596E-05" ixy="-1.32395086473482E-10" ixz="2.69560335696801E-10" iyy="0.000134739848442081" iyz="3.62695515377463E-10" izz="0.000102669008431253" />
+      <inertia ixx="4.13492347432596E-05" ixy="-1.32395086473111E-10" ixz="2.69560335696807E-10" iyy="0.000134739848442081" iyz="3.62695515378734E-10" izz="0.000102669008431253" />
     </inertial>
     <visual>
@@ -189,15 +189,15 @@
     </collision>
   </link>
-  <joint name="right_foot_joint" type="fixed">
-    <origin xyz="-0.014194 0.004875 0.024182" rpy="-1.5581 0 1.5708" />
+  <joint name="right_foot_joint" type="revolute">
+    <origin xyz="-0.0141935477215366 0.00487500000000001 0.0241824978667717" rpy="-1.55807601714472 0 1.5707963267949" />
     <parent link="right_ankle_link" />
     <child link="right_foot_link" />
-    <axis xyz="0 0 0" />
+    <axis xyz="0 1 0" />
   </joint>
   <link name="left_hip_link">
     <inertial>
-      <origin xyz="0.00574384356514769 0.000137242116570632 -0.00899186986767261" rpy="0 0 0" />
-      <mass value="0.027821769923242" />
-      <inertia ixx="5.52363659732332E-06" ixy="2.35404777695923E-22" ixz="9.52912065661088E-22" iyy="5.28896445958682E-06" iyz="-7.01815773253074E-22" izz="2.92981364310441E-06" />
+      <origin xyz="0.00658000217737552 0.000137242116570642 -0.00839934723438571" rpy="0 0 0" />
+      <mass value="0.0278217699232421" />
+      <inertia ixx="5.49976331318411E-06" ixy="-9.79198689602685E-23" ixz="2.47695657405005E-07" iyy="5.28896445958682E-06" iyz="3.54874372163226E-22" izz="2.95368692724363E-06" />
     </inertial>
     <visual>
@@ -218,15 +218,15 @@
   </link>
   <joint name="left_hip" type="revolute">
-    <origin xyz="0.0005 0.015 -0.02" rpy="3.1416 1.3958 1.5708" />
+    <origin xyz="0.0005 0.015 -0.02" rpy="-3.1416 1.3958 1.5708" />
     <parent link="base_link" />
     <child link="left_hip_link" />
     <axis xyz="0 1 0" />
-    <limit lower="-3.0" upper="3.0" effort="1000" velocity="3.0" />
+    <limit lower="-6.28" upper="6.28" effort="1.0" velocity="1.0" />
   </joint>
   <link name="left_thigh_link">
     <inertial>
-      <origin xyz="0.000483541080447515 -1.38777878078145E-17 -0.0288011243914165" rpy="0 0 0" />
+      <origin xyz="-0.00637969318425013 -0.00283659528954072 -0.0290578305835431" rpy="0 0 0" />
       <mass value="0.0440662654824574" />
-      <inertia ixx="6.99871657924005E-06" ixy="-1.30252055807653E-21" ixz="-6.60751594534272E-07" iyy="5.83167629890069E-06" iyz="1.22954384106141E-21" izz="4.6055287326144E-06" />
+      <inertia ixx="6.54856398809019E-06" ixy="-7.39654858335863E-22" ixz="-1.14510044303001E-06" iyy="5.83167629890068E-06" iyz="1.04933415220832E-21" izz="5.05568132376425E-06" />
     </inertial>
     <visual>
@@ -247,15 +247,15 @@
   </link>
   <joint name="left_thigh" type="revolute">
-    <origin xyz="0.03 0.0005 -0.009" rpy="-1.5708 0 1.4529" />
+    <origin xyz="0.03 0.000500000000000025 -0.00899999999999999" rpy="-1.66622377921866 -0.0112365639127549 1.45394144315434" />
     <parent link="left_hip_link" />
     <child link="left_thigh_link" />
     <axis xyz="0 1 0" />
-    <limit lower="-3.0" upper="3.0" effort="1000" velocity="3.0" />
+    <limit lower="-6.28" upper="6.28" effort="1.0" velocity="1.0" />
   </joint>
   <link name="left_knee_link">
     <inertial>
-      <origin xyz="-0.0159002354975483 -6.76542155630955E-16 -0.0317958284727074" rpy="0 0 0" />
-      <mass value="0.0323717699232421" />
-      <inertia ixx="6.09585578173946E-06" ixy="-9.75086376578192E-22" ixz="-2.57710392869743E-07" iyy="3.93488969546397E-06" iyz="-1.37120055400643E-21" izz="4.60249046725557E-06" />
+      <origin xyz="-0.00305906745507309 0.00809905391845241 -0.0376768599798308" rpy="0 0 0" />
+      <mass value="0.032371769923242" />
+      <inertia ixx="6.10807460004073E-06" ixy="1.54712813311779E-21" ixz="-2.19130526484317E-07" iyy="3.93488969546397E-06" iyz="-4.3145409942224E-22" izz="4.59027164895429E-06" />
     </inertial>
     <visual>
@@ -276,15 +276,15 @@
   </link>
   <joint name="left_knee" type="revolute">
-    <origin xyz="-0.0021501 0 -0.055492" rpy="0 -0.49935 3.1416" />
+    <origin xyz="-0.00220959350099466 0.00526245862891174 -0.0552392606252031" rpy="0 -0.497705180578268 3.14159265358979" />
     <parent link="left_thigh_link" />
     <child link="left_knee_link" />
     <axis xyz="0 1 0" />
-    <limit lower="-3.0" upper="3.0" effort="1000" velocity="3.0" />
+    <limit lower="-6.28" upper="6.28" effort="1.0" velocity="1.0" />
   </joint>
   <link name="left_calf_link">
     <inertial>
-      <origin xyz="-0.00690141207525505 0.00108014351796133 0.0255261573931621" rpy="0 0 0" />
-      <mass value="0.0278217699232421" />
-      <inertia ixx="5.30185932211653E-06" ixy="3.09254745805148E-23" ixz="-5.34769808048693E-08" iyy="2.92981364310441E-06" iyz="-8.94604079450337E-22" izz="5.51074173479362E-06" />
+      <origin xyz="0.00802709092672989 -0.0122882354464416 0.0313335965749465" rpy="0 0 0" />
+      <mass value="0.027821769923242" />
+      <inertia ixx="5.29635191124297E-06" ixy="2.14507048611641E-21" ixz="-4.09762691152125E-08" iyy="2.92981364310441E-06" iyz="-2.04402063045031E-21" izz="5.51624914566717E-06" />
     </inertial>
     <visual>
@@ -305,15 +305,15 @@
   </link>
   <joint name="left_calf" type="revolute">
-    <origin xyz="-0.019869 0 -0.053251" rpy="-3.1416 0.052065 0" />
+    <origin xyz="-0.019606921772563 -0.00526932504594984 -0.053087622052145" rpy="3.14159265358979 0.0519735721777248 0" />
     <parent link="left_knee_link" />
     <child link="left_calf_link" />
     <axis xyz="0 1 0" />
-    <limit lower="-3.0" upper="3.0" effort="1000" velocity="3.0" />
+    <limit lower="-6.28" upper="6.28" effort="1.0" velocity="1.0" />
   </joint>
   <link name="left_ankle_link">
     <inertial>
-      <origin xyz="-0.0136213334288442 -0.00459337841653701 -0.013353320848436" rpy="0 0 0" />
-      <mass value="0.132188114966052" />
-      <inertia ixx="0.000136753876292704" ixy="-5.26733657769073E-10" ixz="-7.25991197394409E-07" iyy="4.22864611143807E-05" iyz="-7.24960113429766E-11" izz="0.000105128445504655" />
+      <origin xyz="-0.0147855757229511 0.0116571953898187 0.00335804641884208" rpy="0 0 0" />
+      <mass value="0.132188110609299" />
+      <inertia ixx="0.000136739212107347" ixy="-5.17416639295474E-10" ixz="-9.9541052353683E-07" iyy="4.22864597822615E-05" iyz="-7.11364598949685E-11" izz="0.000105143111721468" />
     </inertial>
     <visual>
@@ -334,9 +334,9 @@
   </link>
   <joint name="left_ankle" type="revolute">
-    <origin xyz="-0.0087077 -0.0075 0.031846" rpy="1.5708 1.3342 0" />
+    <origin xyz="-0.00894754833494107 -0.00443791749499169 0.0323495945430793" rpy="1.10362324462594 1.37074513400544 -0.475321883468647" />
     <parent link="left_calf_link" />
     <child link="left_ankle_link" />
     <axis xyz="0 1 0" />
-    <limit lower="-3.0" upper="3.0" effort="1000" velocity="3.0" />
+    <limit lower="-6.28" upper="6.28" effort="1.0" velocity="1.0" />
   </joint>
   <link name="left_foot_link">
@@ -344,5 +344,5 @@
       <origin xyz="1.35029760289784E-08 0.0104287918497478 1.17152012257815E-08" rpy="0 0 0" />
       <mass value="0.124551473427286" />
-      <inertia ixx="4.13510775251367E-05" ixy="5.14922415404396E-10" ixz="8.73800926913661E-11" iyy="0.000134748648682341" iyz="1.37529274140502E-10" izz="0.000102674182175629" />
+      <inertia ixx="4.13510775251367E-05" ixy="5.14922415402702E-10" ixz="8.73800926931131E-11" iyy="0.000134748648682341" iyz="1.3752927413542E-10" izz="0.000102674182175629" />
     </inertial>
     <visual>
@@ -362,9 +362,9 @@
     </collision>
   </link>
-  <joint name="left_foot_joint" type="fixed">
+  <joint name="left_foot_joint" type="revolute">
     <origin xyz="-0.0254952367690822 0.0113755745672261 0.00285705310295755" rpy="-0.0314669727072048 0 -1.5707963267949" />
     <parent link="left_ankle_link" />
     <child link="left_foot_link" />
-    <axis xyz="0 0 0" />
+    <axis xyz="0 1 0" />
   </joint>
   <link name="right_arm_link">
@@ -372,5 +372,5 @@
       <origin xyz="-9.99200722162641E-16 0.0259259508257144 -2.15105711021124E-16" rpy="0 0 0" />
       <mass value="0.00763663718201332" />
-      <inertia ixx="2.43758966616897E-06" ixy="2.93020214434485E-22" ixz="4.12200417999712E-09" iyy="2.02189199404243E-06" iyz="5.46092272261234E-23" izz="9.35393567758914E-07" />
+      <inertia ixx="2.43758966616897E-06" ixy="2.99482562970055E-22" ixz="4.12200417999712E-09" iyy="2.02189199404243E-06" iyz="7.19892928033102E-23" izz="9.35393567758914E-07" />
     </inertial>
     <visual>
@@ -391,15 +391,15 @@
   </link>
   <joint name="right_shoulder" type="revolute">
-    <origin xyz="-0.007 -0.026 0.075" rpy="3.1416 -1.5708 0" />
+    <origin xyz="-0.007 -0.026 0.075" rpy="0 -1.5708 0" />
     <parent link="base_link" />
     <child link="right_arm_link" />
     <axis xyz="0 1 0" />
-    <limit lower="-3.0" upper="3.0" effort="1000" velocity="3.0" />
+    <limit lower="-6.28" upper="6.28" effort="1.0" velocity="1.0" />
   </joint>
   <link name="right_arm_upper_link">
     <inertial>
-      <origin xyz="-0.0267099408480544 -5.91540705308091E-16 -0.00839330007950644" rpy="0 0 0" />
+      <origin xyz="-0.0267099408480544 -5.91540705308091E-16 -0.00839330007950642" rpy="0 0 0" />
       <mass value="0.0404127433991118" />
-      <inertia ixx="5.33571477961189E-06" ixy="-3.15155813382704E-22" ixz="-1.56386748236192E-07" iyy="6.27306084712395E-06" iyz="-1.94387443949962E-22" izz="5.78424046197137E-06" />
+      <inertia ixx="5.33571477961189E-06" ixy="-3.15982993995257E-22" ixz="-1.56386748236192E-07" iyy="6.27306084712395E-06" iyz="-1.94387443949962E-22" izz="5.78424046197137E-06" />
     </inertial>
     <visual>
@@ -424,5 +424,5 @@
     <child link="right_arm_upper_link" />
     <axis xyz="0 1 0" />
-    <limit lower="-3.0" upper="3.0" effort="1000" velocity="3.0" />
+    <limit lower="-6.28" upper="6.28" effort="1.0" velocity="1.0" />
   </joint>
   <link name="right_arm_lower_link">
@@ -430,5 +430,5 @@
       <origin xyz="0.0182616337014053 0.00084071649884114 -4.33680868994202E-18" rpy="0 0 0" />
       <mass value="0.0290848600660391" />
-      <inertia ixx="2.72498939319332E-06" ixy="-1.67669592897643E-07" ixz="2.5146290621612E-22" iyy="4.0538898836655E-06" iyz="3.57083530681485E-22" izz="4.64311633086366E-06" />
+      <inertia ixx="2.72498939319332E-06" ixy="-1.67669592897643E-07" ixz="2.38228016415272E-22" iyy="4.0538898836655E-06" iyz="3.55842759762656E-22" izz="4.64311633086366E-06" />
     </inertial>
     <visual>
@@ -453,5 +453,5 @@
     <child link="right_arm_lower_link" />
     <axis xyz="0 1 0" />
-    <limit lower="-3.0" upper="3.0" effort="1000" velocity="3.0" />
+    <limit lower="-6.28" upper="6.28" effort="1.0" velocity="1.0" />
   </joint>
   <link name="right_hand_link">
@@ -477,15 +477,15 @@
     </collision>
   </link>
-  <joint name="right_hand_joint" type="fixed">
+  <joint name="right_hand_joint" type="revolute">
     <origin xyz="0.0269999999999999 0 0" rpy="-1.5707963267949 0 -1.5707963267949" />
     <parent link="right_arm_lower_link" />
     <child link="right_hand_link" />
-    <axis xyz="0 0 0" />
+    <axis xyz="0 1 0" />
   </joint>
   <link name="left_arm_link">
     <inertial>
-      <origin xyz="-7.7715611723761E-16 -0.0259259508257144 3.45209971719385E-16" rpy="0 0 0" />
+      <origin xyz="-7.91033905045424E-16 -0.0259259508257144 3.44342609981396E-16" rpy="0 0 0" />
       <mass value="0.00763663718201333" />
-      <inertia ixx="2.43758966616897E-06" ixy="2.47506888618435E-22" ixz="-4.12200417999841E-09" iyy="2.02189199404244E-06" iyz="1.16991672016122E-22" izz="9.35393567758914E-07" />
+      <inertia ixx="2.43758966616897E-06" ixy="2.4695109171783E-22" ixz="-4.12200417999841E-09" iyy="2.02189199404243E-06" iyz="1.02071912761378E-22" izz="9.35393567758914E-07" />
     </inertial>
     <visual>
@@ -506,15 +506,15 @@
   </link>
   <joint name="left_shoulder" type="revolute">
-    <origin xyz="-0.007 0.026 0.075" rpy="3.1416 -1.5708 0" />
+    <origin xyz="-0.007 0.026 0.075" rpy="3.1416 1.5708 0" />
     <parent link="base_link" />
     <child link="left_arm_link" />
     <axis xyz="0 1 0" />
-    <limit lower="-3.0" upper="3.0" effort="1000" velocity="3.0" />
+    <limit lower="-6.28" upper="6.28" effort="1.0" velocity="1.0" />
   </joint>
   <link name="left_arm_upper_link">
     <inertial>
-      <origin xyz="-0.0267099408480542 -4.86589935011494E-16 -0.00839330007950634" rpy="0 0 0" />
+      <origin xyz="-0.0267099408480541 -4.88324658487471E-16 -0.00839330007950632" rpy="0 0 0" />
       <mass value="0.0404127433991118" />
-      <inertia ixx="5.33571477961189E-06" ixy="8.43724224804088E-22" ixz="-1.56386748236191E-07" iyy="6.27306084712395E-06" iyz="3.66441011360991E-22" izz="5.78424046197137E-06" />
+      <inertia ixx="5.33571477961189E-06" ixy="8.42069863578982E-22" ixz="-1.56386748236191E-07" iyy="6.27306084712395E-06" iyz="3.66027421054715E-22" izz="5.78424046197137E-06" />
     </inertial>
     <visual>
@@ -539,5 +539,5 @@
     <child link="left_arm_upper_link" />
     <axis xyz="0 1 0" />
-    <limit lower="-3.0" upper="3.0" effort="1000" velocity="3.0" />
+    <limit lower="-6.28" upper="6.28" effort="1.0" velocity="1.0" />
   </joint>
   <link name="left_arm_lower_link">
@@ -545,5 +545,5 @@
       <origin xyz="0.0182616337014054 0.000840716498841161 -6.93889390390723E-18" rpy="0 0 0" />
       <mass value="0.0290848600660391" />
-      <inertia ixx="2.72498939319332E-06" ixy="-1.67669592897644E-07" ixz="7.94093388050907E-23" iyy="4.0538898836655E-06" iyz="8.69185878034236E-22" izz="4.64311633086366E-06" />
+      <inertia ixx="2.72498939319332E-06" ixy="-1.67669592897644E-07" ixz="1.05879118406788E-22" iyy="4.0538898836655E-06" iyz="8.67557366203272E-22" izz="4.64311633086366E-06" />
     </inertial>
     <visual>
@@ -568,5 +568,5 @@
     <child link="left_arm_lower_link" />
     <axis xyz="0 1 0" />
-    <limit lower="-3.0" upper="3.0" effort="1000" velocity="3.0" />
+    <limit lower="-6.28" upper="6.28" effort="1.0" velocity="1.0" />
   </joint>
   <link name="left_hand_link">
@@ -574,5 +574,5 @@
       <origin xyz="-0.00274751358458326 0 0.0122930084282204" rpy="0 0 0" />
       <mass value="0.00889972732481043" />
-      <inertia ixx="1.20252640088182E-06" ixy="4.72850042347696E-23" ixz="1.67669592897643E-07" iyy="1.14137172758278E-06" iyz="-5.9557004103818E-23" izz="7.30558007213651E-07" />
+      <inertia ixx="1.20252640088182E-06" ixy="5.63839909728529E-23" ixz="1.67669592897643E-07" iyy="1.14137172758278E-06" iyz="-5.9557004103818E-23" izz="7.30558007213651E-07" />
     </inertial>
     <visual>
@@ -592,15 +592,15 @@
     </collision>
   </link>
-  <joint name="left_hand_joint" type="fixed">
+  <joint name="left_hand_joint" type="revolute">
     <origin xyz="0.0269999999999999 0 0" rpy="-1.5707963267949 0 -1.57079632679489" />
     <parent link="left_arm_lower_link" />
     <child link="left_hand_link" />
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