Commit message: more xacro fixes
Signed-off-by: Curt Meyers <cmeyers@boilerbots.com>

File: ros2/src/k1_description/urdf/k1.xacro (robot description, xacro)
@@ -189,9 +189,9 @@
     </collision>
   </link>
-  <joint name="right_foot_joint" type="revolute">
+  <joint name="right_foot_joint" type="fixed">
     <origin xyz="-0.0141935477215366 0.00487500000000001 0.0241824978667717" rpy="-1.55807601714472 0 1.5707963267949" />
     <parent link="right_ankle_link" />
     <child link="right_foot_link" />
-    <axis xyz="0 1 0" />
+    <axis xyz="0 0 0" />
   </joint>
   <link name="left_hip_link">
@@ -362,9 +362,9 @@
     </collision>
   </link>
-  <joint name="left_foot_joint" type="revolute">
+  <joint name="left_foot_joint" type="fixed">
     <origin xyz="-0.0254952367690822 0.0113755745672261 0.00285705310295755" rpy="-0.0314669727072048 0 -1.5707963267949" />
     <parent link="left_ankle_link" />
     <child link="left_foot_link" />
-    <axis xyz="0 1 0" />
+    <axis xyz="0 0 0" />
   </joint>
   <link name="right_arm_link">
@@ -477,9 +477,9 @@
     </collision>
   </link>
-  <joint name="right_hand_joint" type="revolute">
+  <joint name="right_hand_joint" type="fixed">
     <origin xyz="0.0269999999999999 0 0" rpy="-1.5707963267949 0 -1.5707963267949" />
     <parent link="right_arm_lower_link" />
     <child link="right_hand_link" />
-    <axis xyz="0 1 0" />
+    <axis xyz="0 0 0" />
   </joint>
   <link name="left_arm_link">
@@ -592,9 +592,9 @@
     </collision>
   </link>
-  <joint name="left_hand_joint" type="revolute">
+  <joint name="left_hand_joint" type="fixed">
     <origin xyz="0.0269999999999999 0 0" rpy="-1.5707963267949 0 -1.57079632679489" />
     <parent link="left_arm_lower_link" />
     <child link="left_hand_link" />
-    <axis xyz="0 1 0" />
+    <axis xyz="0 0 0" />
   </joint>
   <link name="head_link">

Commit message: Small joint adjustments to get things straight.
Signed-off-by: Curt Meyers <cmeyers@boilerbots.com>

File: ros2/src/k1_description/urdf/k1.xacro (robot description, xacro)
@@ -45,5 +45,5 @@
   </link>
   <joint name="right_hip" type="revolute">
-    <origin xyz="0.0005 -0.015 -0.02" rpy="-3.1416 0 1.5708" />
+    <origin xyz="0.0005 -0.015 -0.02" rpy="-3.1416 0.03 1.5708" />
     <parent link="base_link" />
     <child link="right_hip_link" />
@@ -218,5 +218,5 @@
   </link>
   <joint name="left_hip" type="revolute">
-    <origin xyz="0.0005 0.015 -0.02" rpy="-3.1416 1.3958 1.5708" />
+    <origin xyz="0.0005 0.015 -0.02" rpy="-3.1416 1.4258 1.5708" />
     <parent link="base_link" />
     <child link="left_hip_link" />
@@ -247,5 +247,5 @@
   </link>
   <joint name="left_thigh" type="revolute">
-    <origin xyz="0.03 0.000500000000000025 -0.00899999999999999" rpy="-1.66622377921866 -0.0112365639127549 1.45394144315434" />
+    <origin xyz="0.03 0.000500000000000025 -0.00899999999999999" rpy="-1.66622377921866 -0.0112365639127549 1.75394144315434" />
     <parent link="left_hip_link" />
     <child link="left_thigh_link" />
@@ -391,8 +391,8 @@
   </link>
   <joint name="right_shoulder" type="revolute">
-    <origin xyz="-0.007 -0.026 0.075" rpy="0 -1.5708 0" />
+    <origin xyz="-0.007 -0.026 0.075" rpy="3.1416 -1.5708 0" />
     <parent link="base_link" />
     <child link="right_arm_link" />
-    <axis xyz="0 1 0" />
+    <axis xyz="0 -1 0" />
     <limit lower="-6.28" upper="6.28" effort="1.0" velocity="1.0" />
   </joint>
@@ -506,8 +506,8 @@
   </link>
   <joint name="left_shoulder" type="revolute">
-    <origin xyz="-0.007 0.026 0.075" rpy="3.1416 1.5708 0" />
+    <origin xyz="-0.007 0.026 0.075" rpy="3.1416 -1.5708 0" />
     <parent link="base_link" />
     <child link="left_arm_link" />
-    <axis xyz="0 1 0" />
+    <axis xyz="0 -1 0" />
     <limit lower="-6.28" upper="6.28" effort="1.0" velocity="1.0" />
   </joint>
@@ -624,5 +624,5 @@
     <parent link="base_link" />
     <child link="head_link" />
-    <axis xyz="0 -1 0" />
+    <axis xyz="0 1 0" />
     <limit lower="-6.28" upper="6.28" effort="1.0" velocity="1.0" />
   </joint>

Commit message: Attempting to flip shoulder rotations.
Signed-off-by: Curt Meyers <cmeyers@boilerbots.com>

File: ros2/src/k1_description/urdf/k1.xacro (robot description, xacro)
@@ -394,5 +394,5 @@
     <parent link="base_link" />
     <child link="right_arm_link" />
-    <axis xyz="0 -1 0" />
+    <axis xyz="0 1 0" />
     <limit lower="-6.28" upper="6.28" effort="1.0" velocity="1.0" />
   </joint>
@@ -420,5 +420,5 @@
   </link>
   <joint name="right_upper" type="revolute">
-    <origin xyz="0 0.0350000000000004 0" rpy="-1.56989921107132 -0.00259316215202615 -0.33306656840474" />
+    <origin xyz="0 0.0350000000000004 0" rpy="1.56989921107132 -0.00259316215202615 -0.33306656840474" />
     <parent link="right_arm_link" />
     <child link="right_arm_upper_link" />
@@ -509,5 +509,5 @@
     <parent link="base_link" />
     <child link="left_arm_link" />
-    <axis xyz="0 -1 0" />
+    <axis xyz="0 1 0" />
     <limit lower="-6.28" upper="6.28" effort="1.0" velocity="1.0" />
   </joint>
@@ -535,5 +535,5 @@
   </link>
   <joint name="left_arm_upper" type="revolute">
-    <origin xyz="0 -0.0350000000000004 0" rpy="1.57169344251847 0.00259316215202667 0.33306656840474" />
+    <origin xyz="0 -0.0350000000000004 0" rpy="-1.57169344251847 0.00259316215202667 0.33306656840474" />
     <parent link="left_arm_link" />
     <child link="left_arm_upper_link" />
@@ -600,5 +600,5 @@
   <link name="head_link">
     <inertial>
-      <origin xyz="-5.27015314794523E-07 -0.0192636340735728 1.77662602571516E-05" rpy="0 0 0" />
+      <origin xyz="-5.27015314794523E-07 -0.0192636340735728 -1.77662602571516E-05" rpy="0 0 0" />
       <mass value="0.0901518210219852" />
       <inertia ixx="3.42226307311124E-05" ixy="-4.62380615190642E-10" ixz="-1.35489424526232E-09" iyy="3.57923710083382E-05" iyz="-6.15798115932379E-09" izz="2.41005619280376E-05" />
@@ -621,8 +621,8 @@
   </link>
   <joint name="head" type="revolute">
-    <origin xyz="-0.011 0 0.086" rpy="-1.5707963267949 0 1.5707963267949" />
+    <origin xyz="-0.011 0 0.086" rpy="1.5707963267949 0 1.5707963267949" />
     <parent link="base_link" />
     <child link="head_link" />
-    <axis xyz="0 1 0" />
+    <axis xyz="0 -1 0" />
     <limit lower="-6.28" upper="6.28" effort="1.0" velocity="1.0" />
   </joint>

Commit message: tweak the right shoulder Signed-off-by: Curt Meyers <cmeyers@boilerbots.com>

File: ros2/src/k1_description/urdf/k1.xacro (robot description, xacro)
@@ -420,5 +420,5 @@
   </link>
   <joint name="right_upper" type="revolute">
-    <origin xyz="0 0.0350000000000004 0" rpy="1.56989921107132 -0.00259316215202615 -0.33306656840474" />
+    <origin xyz="0 -0.0350000000000004 0" rpy="1.56989921107132 0.00259316215202615 0.33306656840474" />
     <parent link="right_arm_link" />
     <child link="right_arm_upper_link" />
@@ -624,5 +624,5 @@
     <parent link="base_link" />
     <child link="head_link" />
-    <axis xyz="0 -1 0" />
+    <axis xyz="0 1 0" />
     <limit lower="-6.28" upper="6.28" effort="1.0" velocity="1.0" />
   </joint>
@@ -650,5 +650,5 @@
   </link>
   <joint name="face_joint" type="fixed">
-    <origin xyz="0 0 0" rpy="3.14159265358979 0 0" />
+    <origin xyz="0 0 0" rpy="0 0 0" />
     <parent link="head_link" />
     <child link="face_link" />

Commit message: Tweak the shoulder joint positions
Signed-off-by: Curt Meyers <cmeyers@boilerbots.com>

File: ros2/src/k1_description/urdf/k1.xacro (robot description, xacro)
@@ -420,5 +420,5 @@
   </link>
   <joint name="right_upper" type="revolute">
-    <origin xyz="0 -0.0350000000000004 0" rpy="1.56989921107132 0.00259316215202615 0.33306656840474" />
+    <origin xyz="0 0.0350000000000004 0" rpy="1.56989921107132 0.00259316215202615 0.23306656840474" />
     <parent link="right_arm_link" />
     <child link="right_arm_upper_link" />
@@ -535,5 +535,5 @@
   </link>
   <joint name="left_arm_upper" type="revolute">
-    <origin xyz="0 -0.0350000000000004 0" rpy="-1.57169344251847 0.00259316215202667 0.33306656840474" />
+    <origin xyz="0 -0.0350000000000004 0" rpy="-1.57169344251847 0.00259316215202667 -0.10306656840474" />
     <parent link="left_arm_link" />
     <child link="left_arm_upper_link" />

Commit message: reverse right shoulder Signed-off-by: Curt Meyers <cmeyers@boilerbots.com>

File: ros2/src/k1_description/urdf/k1.xacro (robot description, xacro)
@@ -394,5 +394,5 @@
     <parent link="base_link" />
     <child link="right_arm_link" />
-    <axis xyz="0 1 0" />
+    <axis xyz="0 -1 0" />
     <limit lower="-6.28" upper="6.28" effort="1.0" velocity="1.0" />
   </joint>

Commit message: Try again on the joints Signed-off-by: Curt Meyers <cmeyers@boilerbots.com>

File: ros2/src/k1_description/urdf/k1.xacro (robot description, xacro)
@@ -391,5 +391,5 @@
   </link>
   <joint name="right_shoulder" type="revolute">
-    <origin xyz="-0.007 -0.026 0.075" rpy="3.1416 -1.5708 0" />
+    <origin xyz="-0.007 -0.026 0.075" rpy="3.1416 1.5708 0" />
     <parent link="base_link" />
     <child link="right_arm_link" />
@@ -420,5 +420,5 @@
   </link>
   <joint name="right_upper" type="revolute">
-    <origin xyz="0 0.0350000000000004 0" rpy="1.56989921107132 0.00259316215202615 0.23306656840474" />
+    <origin xyz="0 0.0350000000000004 0" rpy="1.56989921107132 0.00259316215202615 3.54" />
     <parent link="right_arm_link" />
     <child link="right_arm_upper_link" />
@@ -449,8 +449,8 @@
   </link>
   <joint name="right_arm_lower" type="revolute">
-    <origin xyz="-0.0667804560220959 0 -0.0209850111622641" rpy="1.5864967516128 0.304075688258208 -3.0891987069566" />
+    <origin xyz="-0.0667804560220959 0 -0.0209850111622641" rpy="-1.5864967516128 0.304075688258208 3.0891987069566" />
     <parent link="right_arm_upper_link" />
     <child link="right_arm_lower_link" />
-    <axis xyz="0 1 0" />
+    <axis xyz="0 -1 0" />
     <limit lower="-6.28" upper="6.28" effort="1.0" velocity="1.0" />
   </joint>
