Commit message: Huge change, new model
All new and improve URDF.
Hopefully got the origins in the right spots.
Fixed joint naming consistencies.

Left arm still raised.

Signed-off-by: Curt Meyers <cmeyers@boilerbots.com>

File: ros2/src/k1_description/urdf/k1.xacro (robot description, xacro)
@@ -1,22 +1,22 @@
-<robot name="k1_with_hands">
+<robot name="k1">
   <link name="base_link">
     <inertial>
-      <origin xyz="-2.7485E-18 -4.6195E-19 0.047092" rpy="0 0 0" />
+      <origin xyz="-4.61950778389125E-19 2.73283908536959E-18 0.0470916230366492" rpy="0 0 0" />
       <mass value="0.2292" />
-      <inertia ixx="0.00022679" ixy="-3.7705E-21" ixz="-1.2088E-21" iyy="0.00015896" iyz="-2.7674E-21" izz="0.00012895" />
-    </inertial>
-    <visual>
-      <origin xyz="0 0 0" rpy="0 0 0" />
-      <geometry>
-        <mesh filename="package://k1_description/meshes/visual/base_link.STL" />
-      </geometry>
-      <material name="">
-        <color rgba="0.79216 0.81961 0.93333 1" />
-      </material>
-    </visual>
-    <collision>
-      <origin xyz="0 0 0" rpy="0 0 0" />
-      <geometry>
-        <mesh filename="package://k1_description/meshes/collision/base_link.STL" />
+      <inertia ixx="0.00015895767591623" ixy="3.7704942585474E-21" ixz="-2.14051822428277E-21" iyy="0.00022678767591623" iyz="1.20880355025952E-21" izz="0.00012895" />
+    </inertial>
+    <visual>
+      <origin xyz="0 0 0" rpy="0 0 0" />
+      <geometry>
+        <mesh filename="package://robot/meshes/base_link.STL" />
+      </geometry>
+      <material name="">
+        <color rgba="0.792156862745098 0.819607843137255 0.933333333333333 1" />
+      </material>
+    </visual>
+    <collision>
+      <origin xyz="0 0 0" rpy="0 0 0" />
+      <geometry>
+        <mesh filename="package://robot/meshes/base_link.STL" />
       </geometry>
     </collision>
@@ -24,588 +24,460 @@
   <link name="right_hip_link">
     <inertial>
-      <origin xyz="-0.0091910773470667 0.000137242116570623 0.00686156682154296" rpy="0 0 0" />
+      <origin xyz="0.00940359621738448 -0.000137242116570632 0.00656729626457146" rpy="0 0 0" />
       <mass value="0.027821769923242" />
-      <inertia ixx="2.93241080676327E-06" ixy="5.41152994005165E-22" ixz="8.20355865167775E-08" iyy="5.28896445958682E-06" iyz="-5.59192783257843E-22" izz="5.52103943366446E-06" />
-    </inertial>
-    <visual>
-      <origin xyz="0 0 0" rpy="0 0 0" />
-      <geometry>
-        <mesh filename="package://k1_description/meshes/visual/right_hip_link.STL" />
-      </geometry>
-      <material name="">
-        <color rgba="0.250980392156863 0.250980392156863 0.250980392156863 1" />
-      </material>
-    </visual>
-    <collision>
-      <origin xyz="0 0 0" rpy="0 0 0" />
-      <geometry>
-        <mesh filename="package://k1_description/meshes/collision/right_hip_link.STL" />
-      </geometry>
-    </collision>
-  </link>
-  <joint name="right_hip" type="revolute">
-    <origin xyz="0.0005 -0.015 -0.02" rpy="-3.1416 0.03 1.5708" />
+      <inertia ixx="2.92981364310441E-06" ixy="4.30908198288843E-22" ixz="6.28657265540301E-22" iyy="5.28896445958682E-06" iyz="9.46658009525752E-23" izz="5.52363659732332E-06" />
+    </inertial>
+    <visual>
+      <origin xyz="0 0 0" rpy="0 0 0" />
+      <geometry>
+        <mesh filename="package://robot/meshes/right_hip_link.STL" />
+      </geometry>
+      <material name="">
+        <color rgba="0.250980392156863 0.250980392156863 0.250980392156863 1" />
+      </material>
+    </visual>
+    <collision>
+      <origin xyz="0 0 0" rpy="0 0 0" />
+      <geometry>
+        <mesh filename="package://robot/meshes/right_hip_link.STL" />
+      </geometry>
+    </collision>
+  </link>
+  <joint name="right_hip_joint" type="continuous">
+    <origin xyz="-0.015 -0.000499999999999993 -0.02" rpy="-3.14159265358979 0.0316484172966858 -3.14159265358979" />
     <parent link="base_link" />
     <child link="right_hip_link" />
     <axis xyz="0 1 0" />
-    <limit lower="-6.28" upper="6.28" effort="1.0" velocity="3.0" />
   </joint>
   <link name="right_thigh_link">
     <inertial>
-      <origin xyz="0.000483541080447617 -1.04083408558608E-17 0.0288011243914165" rpy="0 0 0" />
-      <mass value="0.0440662654824575" />
-      <inertia ixx="6.99871657924006E-06" ixy="2.48488152353851E-23" ixz="6.60751594534264E-07" iyy="5.83167629890069E-06" iyz="-2.58865577893623E-22" izz="4.6055287326144E-06" />
-    </inertial>
-    <visual>
-      <origin xyz="0 0 0" rpy="0 0 0" />
-      <geometry>
-        <mesh filename="package://k1_description/meshes/visual/right_thigh_link.STL" />
-      </geometry>
-      <material name="">
-        <color rgba="0.250980392156863 0.250980392156863 0.250980392156863 1" />
-      </material>
-    </visual>
-    <collision>
-      <origin xyz="0 0 0" rpy="0 0 0" />
-      <geometry>
-        <mesh filename="package://k1_description/meshes/collision/right_thigh_link.STL" />
-      </geometry>
-    </collision>
-  </link>
-  <joint name="right_thigh" type="revolute">
-    <origin xyz="-0.00945051849090369 0.000499999999999996 0.0333157275209935" rpy="0.0316585832535403 0.0253385921253171 1.57159869279353" />
+      <origin xyz="-0.000246681744016047 -3.46944695195361E-18 0.0288041268970871" rpy="0 0 0" />
+      <mass value="0.0440662654824574" />
+      <inertia ixx="6.96369137755179E-06" ixy="4.38207832004734E-22" ixz="7.20546870045399E-07" iyy="5.83167629890068E-06" iyz="-4.71683349965899E-24" izz="4.64055393430265E-06" />
+    </inertial>
+    <visual>
+      <origin xyz="0 0 0" rpy="0 0 0" />
+      <geometry>
+        <mesh filename="package://robot/meshes/right_thigh_link.STL" />
+      </geometry>
+      <material name="">
+        <color rgba="0.250980392156863 0.250980392156863 0.250980392156863 1" />
+      </material>
+    </visual>
+    <collision>
+      <origin xyz="0 0 0" rpy="0 0 0" />
+      <geometry>
+        <mesh filename="package://robot/meshes/right_thigh_link.STL" />
+      </geometry>
+    </collision>
+  </link>
+  <joint name="right_thigh_joint" type="continuous">
+    <origin xyz="0.0105 -0.000499999999999989 0.033" rpy="0 0.0253512899928625 -1.5707963267949" />
     <parent link="right_hip_link" />
     <child link="right_thigh_link" />
     <axis xyz="0 1 0" />
-    <limit lower="-6.28" upper="6.28" effort="1.0" velocity="1.0" />
   </joint>
   <link name="right_knee_link">
     <inertial>
-      <origin xyz="-0.0178121084477415 3.81639164714898E-17 0.0307655812522569" rpy="0 0 0" />
+      <origin xyz="0.0355383336616086 -3.12250225675825E-17 -0.000905007016273815" rpy="0 0 0" />
       <mass value="0.032371769923242" />
-      <inertia ixx="6.0588731794123E-06" ixy="-3.78363821203638E-22" ixz="3.46807539238869E-07" iyy="3.93488969546397E-06" iyz="4.20940815551816E-22" izz="4.63947306958273E-06" />
-    </inertial>
-    <visual>
-      <origin xyz="0 0 0" rpy="0 0 0" />
-      <geometry>
-        <mesh filename="package://k1_description/meshes/visual/right_knee_link.STL" />
-      </geometry>
-      <material name="">
-        <color rgba="0.752941176470588 1 1 1" />
-      </material>
-    </visual>
-    <collision>
-      <origin xyz="0 0 0" rpy="0 0 0" />
-      <geometry>
-        <mesh filename="package://k1_description/meshes/collision/right_knee_link.STL" />
-      </geometry>
-    </collision>
-  </link>
-  <joint name="right_knee" type="revolute">
-    <origin xyz="-0.00215005179923145 0 0.0554917017754941" rpy="0 0.499346721680126 -3.14159265358979" />
+      <inertia ixx="4.67335720190332E-06" ixy="7.12136216752866E-22" ixz="-4.08928448493292E-07" iyy="3.93488969546397E-06" iyz="-6.52115381615019E-22" izz="6.0249890470917E-06" />
+    </inertial>
+    <visual>
+      <origin xyz="0 0 0" rpy="0 0 0" />
+      <geometry>
+        <mesh filename="package://robot/meshes/right_knee_link.STL" />
+      </geometry>
+      <material name="">
+        <color rgba="0.752941176470588 1 1 1" />
+      </material>
+    </visual>
+    <collision>
+      <origin xyz="0 0 0" rpy="0 0 0" />
+      <geometry>
+        <mesh filename="package://robot/meshes/right_knee_link.STL" />
+      </geometry>
+    </collision>
+  </link>
+  <joint name="right_knee_joint" type="continuous">
+    <origin xyz="-0.00355599647142655 0 0.055419370059348" rpy="-3.14159265358978 -1.54544503680202 3.14159265358978" />
     <parent link="right_thigh_link" />
     <child link="right_knee_link" />
     <axis xyz="0 1 0" />
-    <limit lower="-6.28" upper="6.28" effort="1.0" velocity="1.0" />
   </joint>
   <link name="right_calf_link">
     <inertial>
-      <origin xyz="-0.00958197752831114 0.00108014351796196 -0.0246454845060883" rpy="0 0 0" />
-      <mass value="0.0278217699232421" />
-      <inertia ixx="5.31556206114482E-06" ixy="1.0431771588901E-21" ixz="7.43927658286799E-08" iyy="2.92981364310441E-06" iyz="-2.7149420750487E-22" izz="5.49703899576533E-06" />
-    </inertial>
-    <visual>
-      <origin xyz="0 0 0" rpy="0 0 0" />
-      <geometry>
-        <mesh filename="package://k1_description/meshes/visual/right_calf_link.STL" />
-      </geometry>
-      <material name="">
-        <color rgba="0.752941176470588 1 1 1" />
-      </material>
-    </visual>
-    <collision>
-      <origin xyz="0 0 0" rpy="0 0 0" />
-      <geometry>
-        <mesh filename="package://k1_description/meshes/collision/right_calf_link.STL" />
-      </geometry>
-    </collision>
-  </link>
-  <joint name="right_calf" type="revolute">
-    <origin xyz="-0.0230838749026589 0 0.0519386898416303" rpy="3.14159265358979 -0.113165928627979 0" />
+      <origin xyz="0.0264395340671427 0.00108014351796196 0.000406495024938089" rpy="0 0 0" />
+      <mass value="0.027821769923242" />
+      <inertia ixx="5.52320669558642E-06" ixy="3.31056529427015E-22" ixz="1.00349959696259E-08" iyy="2.9298136431044E-06" iyz="3.62681967144928E-23" izz="5.28939436132371E-06" />
+    </inertial>
+    <visual>
+      <origin xyz="0 0 0" rpy="0 0 0" />
+      <geometry>
+        <mesh filename="package://robot/meshes/right_calf_link.STL" />
+      </geometry>
+      <material name="">
+        <color rgba="0.752941176470588 1 1 1" />
+      </material>
+    </visual>
+    <collision>
+      <origin xyz="0 0 0" rpy="0 0 0" />
+      <geometry>
+        <mesh filename="package://robot/meshes/right_calf_link.STL" />
+      </geometry>
+    </collision>
+  </link>
+  <joint name="right_calf_joint" type="continuous">
+    <origin xyz="0.0566505085564426 0 0.00460572071266819" rpy="0 0 0" />
     <parent link="right_knee_link" />
     <child link="right_calf_link" />
     <axis xyz="0 1 0" />
-    <limit lower="-6.28" upper="6.28" effort="1.0" velocity="1.0" />
   </joint>
   <link name="right_ankle_link">
     <inertial>
-      <origin xyz="-0.0134919017266966 0.00459336693369054 0.0134840145322273" rpy="0 0 0" />
-      <mass value="0.132188163411726" />
-      <inertia ixx="0.000105111740356927" ixy="-2.67854466622726E-10" ixz="4.02982212640105E-07" iyy="4.22846170003843E-05" iyz="1.35813174315733E-10" izz="0.000136756609487253" />
-    </inertial>
-    <visual>
-      <origin xyz="0 0 0" rpy="0 0 0" />
-      <geometry>
-        <mesh filename="package://k1_description/meshes/visual/right_ankle_link.STL" />
-      </geometry>
-      <material name="">
-        <color rgba="0.752941176470588 1 1 1" />
-      </material>
-    </visual>
-    <collision>
-      <origin xyz="0 0 0" rpy="0 0 0" />
-      <geometry>
-        <mesh filename="package://k1_description/meshes/collision/right_ankle_link.STL" />
-      </geometry>
-    </collision>
-  </link>
-  <joint name="right_ankle" type="revolute">
-    <origin xyz="-0.0120513798099409 -0.00749999999999831 -0.0307370174980681" rpy="2.79822593138815 0 -1.5707963267949" />
+      <origin xyz="0.0136623267443019 -0.00459336936624942 0.0133113128666117" rpy="0 0 0" />
+      <mass value="0.132188160242468" />
+      <inertia ixx="0.000105106606233086" ixy="-2.6922058885189E-10" ixz="-3.57117309042543E-10" iyy="4.22846167628333E-05" iyz="-1.31879399966339E-10" izz="0.000136761741778018" />
+    </inertial>
+    <visual>
+      <origin xyz="0 0 0" rpy="0 0 0" />
+      <geometry>
+        <mesh filename="package://robot/meshes/right_ankle_link.STL" />
+      </geometry>
+      <material name="">
+        <color rgba="0.752941176470588 1 1 1" />
+      </material>
+    </visual>
+    <collision>
+      <origin xyz="0 0 0" rpy="0 0 0" />
+      <geometry>
+        <mesh filename="package://robot/meshes/right_ankle_link.STL" />
+      </geometry>
+    </collision>
+  </link>
+  <joint name="right_ankle_joint" type="continuous">
+    <origin xyz="0.0330125603748861 -0.0074999999999983 0.000413349119391304" rpy="1.52798571545966 -0.000544427216642011 1.55808767255617" />
     <parent link="right_calf_link" />
     <child link="right_ankle_link" />
     <axis xyz="0 1 0" />
-    <limit lower="-6.28" upper="6.28" effort="1.0" velocity="1.0" />
-  </joint>
-  <link name="right_foot_link">
-    <inertial>
-      <origin xyz="3.89163107121504E-10 0.0104288935743586 5.67569245074617E-09" rpy="0 0 0" />
-      <mass value="0.124551526229713" />
-      <inertia ixx="4.13492347432596E-05" ixy="-1.32395086473111E-10" ixz="2.69560335696807E-10" iyy="0.000134739848442081" iyz="3.62695515378734E-10" izz="0.000102669008431253" />
-    </inertial>
-    <visual>
-      <origin xyz="0 0 0" rpy="0 0 0" />
-      <geometry>
-        <mesh filename="package://k1_description/meshes/visual/right_foot_link.STL" />
-      </geometry>
-      <material name="">
-        <color rgba="1 1 0.752941176470588 1" />
-      </material>
-    </visual>
-    <collision>
-      <origin xyz="0 0 0" rpy="0 0 0" />
-      <geometry>
-        <mesh filename="package://k1_description/meshes/collision/right_foot_link.STL" />
-      </geometry>
-    </collision>
-  </link>
-  <joint name="right_foot_joint" type="fixed">
-    <origin xyz="-0.0141935477215366 0.00487500000000001 0.0241824978667717" rpy="-1.55807601714472 0 1.5707963267949" />
-    <parent link="right_ankle_link" />
-    <child link="right_foot_link" />
-    <axis xyz="0 0 0" />
   </joint>
   <link name="left_hip_link">
     <inertial>
-      <origin xyz="0.00658000217737552 0.000137242116570642 -0.00839934723438571" rpy="0 0 0" />
-      <mass value="0.0278217699232421" />
-      <inertia ixx="5.49976331318411E-06" ixy="-9.79198689602685E-23" ixz="2.47695657405005E-07" iyy="5.28896445958682E-06" iyz="3.54874372163226E-22" izz="2.95368692724363E-06" />
-    </inertial>
-    <visual>
-      <origin xyz="0 0 0" rpy="0 0 0" />
-      <geometry>
-        <mesh filename="package://k1_description/meshes/visual/left_hip_link.STL" />
-      </geometry>
-      <material name="">
-        <color rgba="0.250980392156863 0.250980392156863 0.250980392156863 1" />
-      </material>
-    </visual>
-    <collision>
-      <origin xyz="0 0 0" rpy="0 0 0" />
-      <geometry>
-        <mesh filename="package://k1_description/meshes/collision/left_hip_link.STL" />
-      </geometry>
-    </collision>
-  </link>
-  <joint name="left_hip" type="revolute">
-    <origin xyz="0.0005 0.015 -0.02" rpy="-3.1416 1.4258 1.5708" />
+      <origin xyz="0.0089918698676726 0.000137242116570587 0.00656729626457131" rpy="0 0 0" />
+      <mass value="0.027821769923242" />
+      <inertia ixx="2.92981364310441E-06" ixy="1.05304755240537E-22" ixz="-6.61744490042422E-22" iyy="5.28896445958682E-06" iyz="1.63447699966183E-22" izz="5.52363659732332E-06" />
+    </inertial>
+    <visual>
+      <origin xyz="0 0 0" rpy="0 0 0" />
+      <geometry>
+        <mesh filename="package://robot/meshes/left_hip_link.STL" />
+      </geometry>
+      <material name="">
+        <color rgba="0.250980392156863 0.250980392156863 0.250980392156863 1" />
+      </material>
+    </visual>
+    <collision>
+      <origin xyz="0 0 0" rpy="0 0 0" />
+      <geometry>
+        <mesh filename="package://robot/meshes/left_hip_link.STL" />
+      </geometry>
+    </collision>
+  </link>
+  <joint name="left_hip_joint" type="continuous">
+    <origin xyz="0.015 -0.000500000000000029 -0.02" rpy="3.14159265358979 -0.0788882616806473 0" />
     <parent link="base_link" />
     <child link="left_hip_link" />
     <axis xyz="0 1 0" />
-    <limit lower="-6.28" upper="6.28" effort="1.0" velocity="1.0" />
   </joint>
   <link name="left_thigh_link">
     <inertial>
-      <origin xyz="-0.00637969318425013 -0.00283659528954072 -0.0290578305835431" rpy="0 0 0" />
-      <mass value="0.0440662654824574" />
-      <inertia ixx="6.54856398809019E-06" ixy="-7.39654858335863E-22" ixz="-1.14510044303001E-06" iyy="5.83167629890068E-06" iyz="1.04933415220832E-21" izz="5.05568132376425E-06" />
-    </inertial>
-    <visual>
-      <origin xyz="0 0 0" rpy="0 0 0" />
-      <geometry>
-        <mesh filename="package://k1_description/meshes/visual/left_thigh_link.STL" />
-      </geometry>
-      <material name="">
-        <color rgba="0.250980392156863 0.250980392156863 0.250980392156863 1" />
-      </material>
-    </visual>
-    <collision>
-      <origin xyz="0 0 0" rpy="0 0 0" />
-      <geometry>
-        <mesh filename="package://k1_description/meshes/collision/left_thigh_link.STL" />
-      </geometry>
-    </collision>
-  </link>
-  <joint name="left_thigh" type="revolute">
-    <origin xyz="0.03 0.000500000000000025 -0.00899999999999999" rpy="-1.66622377921866 -0.0112365639127549 1.75394144315434" />
+      <origin xyz="0.0288011243914165 1.04083408558608E-17 -0.000483541080447512" rpy="0 0 0" />
+      <mass value="0.0440662654824575" />
+      <inertia ixx="4.6055287326144E-06" ixy="1.12360003625057E-21" ixz="-6.60751594534273E-07" iyy="5.83167629890069E-06" iyz="-1.04244405181093E-21" izz="6.99871657924005E-06" />
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