Commit message: Huge change, new model
All new and improve URDF.
Hopefully got the origins in the right spots.
Fixed joint naming consistencies.

Left arm still raised.

Signed-off-by: Curt Meyers <cmeyers@boilerbots.com>

File: ros2/src/k1_moveit/config/k1.ros2_control.xacro (robot description, xacro)
@@ -5,124 +5,127 @@
         <ros2_control name="${name}" type="system">
             <hardware>
-                <!--<plugin>mock_components/GenericSystem</plugin>-->
+                <!-- By default, set up controllers for simulation. This won't work on real hardware -->
+<!--
+                <plugin>mock_components/GenericSystem</plugin>
+-->
                 <plugin>k1_control/RobotSystem</plugin>
                 <param name="device">/dev/ttyAMA0</param>
             </hardware>
-            <joint name="left_thigh">
+            <joint name="right_hip_joint">
                 <command_interface name="position"/>
                 <state_interface name="position">
-                  <param name="initial_value">${initial_positions['left_thigh']}</param>
+                  <param name="initial_value">${initial_positions['right_hip_joint']}</param>
                 </state_interface>
                 <state_interface name="velocity"/>
             </joint>
-            <joint name="left_knee">
+            <joint name="right_thigh_joint">
                 <command_interface name="position"/>
                 <state_interface name="position">
-                  <param name="initial_value">${initial_positions['left_knee']}</param>
+                  <param name="initial_value">${initial_positions['right_thigh_joint']}</param>
                 </state_interface>
                 <state_interface name="velocity"/>
             </joint>
-            <joint name="left_calf">
+            <joint name="right_knee_joint">
                 <command_interface name="position"/>
                 <state_interface name="position">
-                  <param name="initial_value">${initial_positions['left_calf']}</param>
+                  <param name="initial_value">${initial_positions['right_knee_joint']}</param>
                 </state_interface>
                 <state_interface name="velocity"/>
             </joint>
-            <joint name="right_thigh">
+            <joint name="right_calf_joint">
                 <command_interface name="position"/>
                 <state_interface name="position">
-                  <param name="initial_value">${initial_positions['right_thigh']}</param>
+                  <param name="initial_value">${initial_positions['right_calf_joint']}</param>
                 </state_interface>
                 <state_interface name="velocity"/>
             </joint>
-            <joint name="right_knee">
+            <joint name="right_ankle_joint">
                 <command_interface name="position"/>
                 <state_interface name="position">
-                  <param name="initial_value">${initial_positions['right_knee']}</param>
+                  <param name="initial_value">${initial_positions['right_ankle_joint']}</param>
                 </state_interface>
                 <state_interface name="velocity"/>
             </joint>
-            <joint name="right_calf">
+            <joint name="left_hip_joint">
                 <command_interface name="position"/>
                 <state_interface name="position">
-                  <param name="initial_value">${initial_positions['right_calf']}</param>
+                  <param name="initial_value">${initial_positions['left_hip_joint']}</param>
                 </state_interface>
                 <state_interface name="velocity"/>
             </joint>
-            <joint name="left_shoulder">
+            <joint name="left_thigh_joint">
                 <command_interface name="position"/>
                 <state_interface name="position">
-                  <param name="initial_value">${initial_positions['left_shoulder']}</param>
+                  <param name="initial_value">${initial_positions['left_thigh_joint']}</param>
                 </state_interface>
                 <state_interface name="velocity"/>
             </joint>
-            <joint name="right_shoulder">
+            <joint name="left_knee_joint">
                 <command_interface name="position"/>
                 <state_interface name="position">
-                  <param name="initial_value">${initial_positions['right_shoulder']}</param>
+                  <param name="initial_value">${initial_positions['left_knee_joint']}</param>
                 </state_interface>
                 <state_interface name="velocity"/>
             </joint>
-            <joint name="left_hip">
+            <joint name="left_calf_joint">
                 <command_interface name="position"/>
                 <state_interface name="position">
-                  <param name="initial_value">${initial_positions['left_hip']}</param>
+                  <param name="initial_value">${initial_positions['left_calf_joint']}</param>
                 </state_interface>
                 <state_interface name="velocity"/>
             </joint>
-            <joint name="left_ankle">
+            <joint name="left_ankle_joint">
                 <command_interface name="position"/>
                 <state_interface name="position">
-                  <param name="initial_value">${initial_positions['left_ankle']}</param>
+                  <param name="initial_value">${initial_positions['left_ankle_joint']}</param>
                 </state_interface>
                 <state_interface name="velocity"/>
             </joint>
-            <joint name="right_hip">
+            <joint name="right_shoulder_joint">
                 <command_interface name="position"/>
                 <state_interface name="position">
-                  <param name="initial_value">${initial_positions['right_hip']}</param>
+                  <param name="initial_value">${initial_positions['right_shoulder_joint']}</param>
                 </state_interface>
                 <state_interface name="velocity"/>
             </joint>
-            <joint name="right_ankle">
+            <joint name="right_upper_arm_joint">
                 <command_interface name="position"/>
                 <state_interface name="position">
-                  <param name="initial_value">${initial_positions['right_ankle']}</param>
+                  <param name="initial_value">${initial_positions['right_upper_arm_joint']}</param>
                 </state_interface>
                 <state_interface name="velocity"/>
             </joint>
-            <joint name="left_arm_upper">
+            <joint name="right_lower_arm_joint">
                 <command_interface name="position"/>
                 <state_interface name="position">
-                  <param name="initial_value">${initial_positions['left_arm_upper']}</param>
+                  <param name="initial_value">${initial_positions['right_lower_arm_joint']}</param>
                 </state_interface>
                 <state_interface name="velocity"/>
             </joint>
-            <joint name="left_arm_lower">
+            <joint name="left_shoulder_joint">
                 <command_interface name="position"/>
                 <state_interface name="position">
-                  <param name="initial_value">${initial_positions['left_arm_lower']}</param>
+                  <param name="initial_value">${initial_positions['left_shoulder_joint']}</param>
                 </state_interface>
                 <state_interface name="velocity"/>
             </joint>
-            <joint name="right_upper">
+            <joint name="left_upper_arm_joint">
                 <command_interface name="position"/>
                 <state_interface name="position">
-                  <param name="initial_value">${initial_positions['right_upper']}</param>
+                  <param name="initial_value">${initial_positions['left_upper_arm_joint']}</param>
                 </state_interface>
                 <state_interface name="velocity"/>
             </joint>
-            <joint name="right_arm_lower">
+            <joint name="left_lower_arm_joint">
                 <command_interface name="position"/>
                 <state_interface name="position">
-                  <param name="initial_value">${initial_positions['right_arm_lower']}</param>
+                  <param name="initial_value">${initial_positions['left_lower_arm_joint']}</param>
                 </state_interface>
                 <state_interface name="velocity"/>
             </joint>
-            <joint name="head">
+            <joint name="head_joint">
                 <command_interface name="position"/>
                 <state_interface name="position">
-                  <param name="initial_value">${initial_positions['head']}</param>
+                  <param name="initial_value">${initial_positions['head_joint']}</param>
                 </state_interface>
                 <state_interface name="velocity"/>

Commit message: OK, put back meshes
Signed-off-by: Curt Meyers <cmeyers@boilerbots.com>

File: ros2/src/k1_description/urdf/k1.xacro (robot description, xacro)
@@ -9,5 +9,5 @@
       <origin xyz="0 0 0" rpy="0 0 0" />
       <geometry>
-        <mesh filename="package://robot/meshes/base_link.STL" />
+        <mesh filename="package://robot/meshes/visual/base_link.STL" />
       </geometry>
       <material name="">
@@ -18,5 +18,5 @@
       <origin xyz="0 0 0" rpy="0 0 0" />
       <geometry>
-        <mesh filename="package://robot/meshes/base_link.STL" />
+        <mesh filename="package://robot/meshes/collision/base_link.STL" />
       </geometry>
     </collision>
@@ -31,14 +31,14 @@
       <origin xyz="0 0 0" rpy="0 0 0" />
       <geometry>
-        <mesh filename="package://robot/meshes/right_hip_link.STL" />
-      </geometry>
-      <material name="">
-        <color rgba="0.250980392156863 0.250980392156863 0.250980392156863 1" />
-      </material>
-    </visual>
-    <collision>
-      <origin xyz="0 0 0" rpy="0 0 0" />
-      <geometry>
-        <mesh filename="package://robot/meshes/right_hip_link.STL" />
+        <mesh filename="package://robot/meshes/visual/right_hip_link.STL" />
+      </geometry>
+      <material name="">
+        <color rgba="0.250980392156863 0.250980392156863 0.250980392156863 1" />
+      </material>
+    </visual>
+    <collision>
+      <origin xyz="0 0 0" rpy="0 0 0" />
+      <geometry>
+        <mesh filename="package://robot/meshes/collision/right_hip_link.STL" />
       </geometry>
     </collision>
@@ -59,14 +59,14 @@
       <origin xyz="0 0 0" rpy="0 0 0" />
       <geometry>
-        <mesh filename="package://robot/meshes/right_thigh_link.STL" />
-      </geometry>
-      <material name="">
-        <color rgba="0.250980392156863 0.250980392156863 0.250980392156863 1" />
-      </material>
-    </visual>
-    <collision>
-      <origin xyz="0 0 0" rpy="0 0 0" />
-      <geometry>
-        <mesh filename="package://robot/meshes/right_thigh_link.STL" />
+        <mesh filename="package://robot/meshes/visual/right_thigh_link.STL" />
+      </geometry>
+      <material name="">
+        <color rgba="0.250980392156863 0.250980392156863 0.250980392156863 1" />
+      </material>
+    </visual>
+    <collision>
+      <origin xyz="0 0 0" rpy="0 0 0" />
+      <geometry>
+        <mesh filename="package://robot/meshes/collision/right_thigh_link.STL" />
       </geometry>
     </collision>
@@ -87,14 +87,14 @@
       <origin xyz="0 0 0" rpy="0 0 0" />
       <geometry>
-        <mesh filename="package://robot/meshes/right_knee_link.STL" />
-      </geometry>
-      <material name="">
-        <color rgba="0.752941176470588 1 1 1" />
-      </material>
-    </visual>
-    <collision>
-      <origin xyz="0 0 0" rpy="0 0 0" />
-      <geometry>
-        <mesh filename="package://robot/meshes/right_knee_link.STL" />
+        <mesh filename="package://robot/meshes/visual/right_knee_link.STL" />
+      </geometry>
+      <material name="">
+        <color rgba="0.752941176470588 1 1 1" />
+      </material>
+    </visual>
+    <collision>
+      <origin xyz="0 0 0" rpy="0 0 0" />
+      <geometry>
+        <mesh filename="package://robot/meshes/collision/right_knee_link.STL" />
       </geometry>
     </collision>
@@ -115,14 +115,14 @@
       <origin xyz="0 0 0" rpy="0 0 0" />
       <geometry>
-        <mesh filename="package://robot/meshes/right_calf_link.STL" />
-      </geometry>
-      <material name="">
-        <color rgba="0.752941176470588 1 1 1" />
-      </material>
-    </visual>
-    <collision>
-      <origin xyz="0 0 0" rpy="0 0 0" />
-      <geometry>
-        <mesh filename="package://robot/meshes/right_calf_link.STL" />
+        <mesh filename="package://robot/meshes/visual/right_calf_link.STL" />
+      </geometry>
+      <material name="">
+        <color rgba="0.752941176470588 1 1 1" />
+      </material>
+    </visual>
+    <collision>
+      <origin xyz="0 0 0" rpy="0 0 0" />
+      <geometry>
+        <mesh filename="package://robot/meshes/collision/right_calf_link.STL" />
       </geometry>
     </collision>
@@ -143,14 +143,14 @@
       <origin xyz="0 0 0" rpy="0 0 0" />
       <geometry>
-        <mesh filename="package://robot/meshes/right_ankle_link.STL" />
-      </geometry>
-      <material name="">
-        <color rgba="0.752941176470588 1 1 1" />
-      </material>
-    </visual>
-    <collision>
-      <origin xyz="0 0 0" rpy="0 0 0" />
-      <geometry>
-        <mesh filename="package://robot/meshes/right_ankle_link.STL" />
+        <mesh filename="package://robot/meshes/visual/right_ankle_link.STL" />
+      </geometry>
+      <material name="">
+        <color rgba="0.752941176470588 1 1 1" />
+      </material>
+    </visual>
+    <collision>
+      <origin xyz="0 0 0" rpy="0 0 0" />
+      <geometry>
+        <mesh filename="package://robot/meshes/collision/right_ankle_link.STL" />
       </geometry>
     </collision>
@@ -171,14 +171,14 @@
       <origin xyz="0 0 0" rpy="0 0 0" />
       <geometry>
-        <mesh filename="package://robot/meshes/left_hip_link.STL" />
-      </geometry>
-      <material name="">
-        <color rgba="0.250980392156863 0.250980392156863 0.250980392156863 1" />
-      </material>
-    </visual>
-    <collision>
-      <origin xyz="0 0 0" rpy="0 0 0" />
-      <geometry>
-        <mesh filename="package://robot/meshes/left_hip_link.STL" />
+        <mesh filename="package://robot/meshes/visual/left_hip_link.STL" />
+      </geometry>
+      <material name="">
+        <color rgba="0.250980392156863 0.250980392156863 0.250980392156863 1" />
+      </material>
+    </visual>
+    <collision>
+      <origin xyz="0 0 0" rpy="0 0 0" />
+      <geometry>
+        <mesh filename="package://robot/meshes/collision/left_hip_link.STL" />
       </geometry>
     </collision>
@@ -199,14 +199,14 @@
       <origin xyz="0 0 0" rpy="0 0 0" />
       <geometry>
-        <mesh filename="package://robot/meshes/left_thigh_link.STL" />
-      </geometry>
-      <material name="">
-        <color rgba="0.250980392156863 0.250980392156863 0.250980392156863 1" />
-      </material>
-    </visual>
-    <collision>
-      <origin xyz="0 0 0" rpy="0 0 0" />
-      <geometry>
-        <mesh filename="package://robot/meshes/left_thigh_link.STL" />
+        <mesh filename="package://robot/meshes/visual/left_thigh_link.STL" />
+      </geometry>
+      <material name="">
+        <color rgba="0.250980392156863 0.250980392156863 0.250980392156863 1" />
+      </material>
+    </visual>
+    <collision>
+      <origin xyz="0 0 0" rpy="0 0 0" />
+      <geometry>
+        <mesh filename="package://robot/meshes/collision/left_thigh_link.STL" />
       </geometry>
     </collision>
@@ -227,14 +227,14 @@
       <origin xyz="0 0 0" rpy="0 0 0" />
       <geometry>
-        <mesh filename="package://robot/meshes/left_knee_link.STL" />
-      </geometry>
-      <material name="">
-        <color rgba="0.752941176470588 1 1 1" />
-      </material>
-    </visual>
-    <collision>
-      <origin xyz="0 0 0" rpy="0 0 0" />
-      <geometry>
-        <mesh filename="package://robot/meshes/left_knee_link.STL" />
+        <mesh filename="package://robot/meshes/visual/left_knee_link.STL" />
+      </geometry>
+      <material name="">
+        <color rgba="0.752941176470588 1 1 1" />
+      </material>
+    </visual>
+    <collision>
+      <origin xyz="0 0 0" rpy="0 0 0" />
+      <geometry>
+        <mesh filename="package://robot/meshes/collision/left_knee_link.STL" />
       </geometry>
     </collision>
@@ -255,14 +255,14 @@
       <origin xyz="0 0 0" rpy="0 0 0" />
       <geometry>
-        <mesh filename="package://robot/meshes/left_calf_link.STL" />
-      </geometry>
-      <material name="">
-        <color rgba="0.752941176470588 1 1 1" />
-      </material>
-    </visual>
-    <collision>
-      <origin xyz="0 0 0" rpy="0 0 0" />
-      <geometry>
-        <mesh filename="package://robot/meshes/left_calf_link.STL" />
+        <mesh filename="package://robot/meshes/visual/left_calf_link.STL" />
+      </geometry>
+      <material name="">
+        <color rgba="0.752941176470588 1 1 1" />
+      </material>
+    </visual>
+    <collision>
+      <origin xyz="0 0 0" rpy="0 0 0" />
+      <geometry>
+        <mesh filename="package://robot/meshes/collision/left_calf_link.STL" />
       </geometry>
     </collision>
@@ -283,14 +283,14 @@
       <origin xyz="0 0 0" rpy="0 0 0" />
       <geometry>
-        <mesh filename="package://robot/meshes/left_ankle_link.STL" />
-      </geometry>
-      <material name="">
-        <color rgba="0.752941176470588 1 1 1" />
-      </material>
-    </visual>
-    <collision>
-      <origin xyz="0 0 0" rpy="0 0 0" />
-      <geometry>
-        <mesh filename="package://robot/meshes/left_ankle_link.STL" />
+        <mesh filename="package://robot/meshes/visual/left_ankle_link.STL" />
+      </geometry>
+      <material name="">
+        <color rgba="0.752941176470588 1 1 1" />
+      </material>
+    </visual>
+    <collision>
+      <origin xyz="0 0 0" rpy="0 0 0" />
+      <geometry>
+        <mesh filename="package://robot/meshes/collision/left_ankle_link.STL" />
       </geometry>
     </collision>
@@ -311,14 +311,14 @@
       <origin xyz="0 0 0" rpy="0 0 0" />
       <geometry>
-        <mesh filename="package://robot/meshes/right_shoulder_link.STL" />
-      </geometry>
-      <material name="">
-        <color rgba="0.752941176470588 1 1 1" />
-      </material>
-    </visual>
-    <collision>
-      <origin xyz="0 0 0" rpy="0 0 0" />
-      <geometry>
-        <mesh filename="package://robot/meshes/right_shoulder_link.STL" />
+        <mesh filename="package://robot/meshes/visual/right_shoulder_link.STL" />
+      </geometry>
+      <material name="">
+        <color rgba="0.752941176470588 1 1 1" />
+      </material>
+    </visual>
+    <collision>
+      <origin xyz="0 0 0" rpy="0 0 0" />
+      <geometry>
+        <mesh filename="package://robot/meshes/collision/right_shoulder_link.STL" />
       </geometry>
     </collision>
@@ -339,14 +339,14 @@
       <origin xyz="0 0 0" rpy="0 0 0" />
       <geometry>
-        <mesh filename="package://robot/meshes/right_upper_arm_link.STL" />
-      </geometry>
-      <material name="">
-        <color rgba="0.250980392156863 0.250980392156863 0.250980392156863 1" />
-      </material>
-    </visual>
-    <collision>
-      <origin xyz="0 0 0" rpy="0 0 0" />
-      <geometry>
-        <mesh filename="package://robot/meshes/right_upper_arm_link.STL" />
+        <mesh filename="package://robot/meshes/visual/right_upper_arm_link.STL" />
+      </geometry>
+      <material name="">
+        <color rgba="0.250980392156863 0.250980392156863 0.250980392156863 1" />
+      </material>
+    </visual>
+    <collision>
+      <origin xyz="0 0 0" rpy="0 0 0" />
+      <geometry>
+        <mesh filename="package://robot/meshes/collision/right_upper_arm_link.STL" />
       </geometry>
     </collision>
@@ -367,14 +367,14 @@
       <origin xyz="0 0 0" rpy="0 0 0" />
       <geometry>
-        <mesh filename="package://robot/meshes/right_lower_arm_link.STL" />
-      </geometry>
-      <material name="">
-        <color rgba="0.250980392156863 0.250980392156863 0.250980392156863 1" />
-      </material>
-    </visual>
-    <collision>
-      <origin xyz="0 0 0" rpy="0 0 0" />
-      <geometry>
-        <mesh filename="package://robot/meshes/right_lower_arm_link.STL" />
+        <mesh filename="package://robot/meshes/visual/right_lower_arm_link.STL" />
+      </geometry>
+      <material name="">
+        <color rgba="0.250980392156863 0.250980392156863 0.250980392156863 1" />
+      </material>
+    </visual>
+    <collision>
+      <origin xyz="0 0 0" rpy="0 0 0" />
+      <geometry>
+        <mesh filename="package://robot/meshes/collision/right_lower_arm_link.STL" />
       </geometry>
     </collision>
@@ -395,14 +395,14 @@
       <origin xyz="0 0 0" rpy="0 0 0" />
       <geometry>
-        <mesh filename="package://robot/meshes/left_shoulder_link.STL" />
-      </geometry>
-      <material name="">
-        <color rgba="0.752941176470588 1 1 1" />
-      </material>
-    </visual>
-    <collision>
-      <origin xyz="0 0 0" rpy="0 0 0" />
-      <geometry>
-        <mesh filename="package://robot/meshes/left_shoulder_link.STL" />
+        <mesh filename="package://robot/meshes/visual/left_shoulder_link.STL" />
+      </geometry>
+      <material name="">
+        <color rgba="0.752941176470588 1 1 1" />
+      </material>
+    </visual>
+    <collision>
+      <origin xyz="0 0 0" rpy="0 0 0" />
+      <geometry>
+        <mesh filename="package://robot/meshes/collision/left_shoulder_link.STL" />
       </geometry>
     </collision>
@@ -423,14 +423,14 @@
       <origin xyz="0 0 0" rpy="0 0 0" />
       <geometry>
-        <mesh filename="package://robot/meshes/left_upper_arm_link.STL" />
-      </geometry>
-      <material name="">
-        <color rgba="0.250980392156863 0.250980392156863 0.250980392156863 1" />
-      </material>
-    </visual>
-    <collision>
-      <origin xyz="0 0 0" rpy="0 0 0" />
-      <geometry>
-        <mesh filename="package://robot/meshes/left_upper_arm_link.STL" />
+        <mesh filename="package://robot/meshes/visual/left_upper_arm_link.STL" />
+      </geometry>
+      <material name="">
+        <color rgba="0.250980392156863 0.250980392156863 0.250980392156863 1" />
+      </material>
+    </visual>
+    <collision>
+      <origin xyz="0 0 0" rpy="0 0 0" />
+      <geometry>
+        <mesh filename="package://robot/meshes/collision/left_upper_arm_link.STL" />
       </geometry>
     </collision>
@@ -451,14 +451,14 @@
       <origin xyz="0 0 0" rpy="0 0 0" />
       <geometry>
-        <mesh filename="package://robot/meshes/left_lower_arm_link.STL" />
-      </geometry>
-      <material name="">
-        <color rgba="0.250980392156863 0.250980392156863 0.250980392156863 1" />
-      </material>
-    </visual>
-    <collision>
-      <origin xyz="0 0 0" rpy="0 0 0" />
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