Commit message: Fixed mesh problems
Signed-off-by: Curt Meyers <cmeyers@boilerbots.com>

File: ros2/src/k1_description/urdf/k1.xacro (robot description, xacro)
@@ -9,5 +9,5 @@
       <origin xyz="0 0 0" rpy="0 0 0" />
       <geometry>
-        <mesh filename="package://robot/meshes/visual/base_link.STL" />
+        <mesh filename="package://k1_description/meshes/visual/base_link.STL" />
       </geometry>
       <material name="">
@@ -18,5 +18,5 @@
       <origin xyz="0 0 0" rpy="0 0 0" />
       <geometry>
-        <mesh filename="package://robot/meshes/collision/base_link.STL" />
+        <mesh filename="package://k1_description/meshes/collision/base_link.STL" />
       </geometry>
     </collision>
@@ -31,14 +31,14 @@
       <origin xyz="0 0 0" rpy="0 0 0" />
       <geometry>
-        <mesh filename="package://robot/meshes/visual/right_hip_link.STL" />
-      </geometry>
-      <material name="">
-        <color rgba="0.250980392156863 0.250980392156863 0.250980392156863 1" />
-      </material>
-    </visual>
-    <collision>
-      <origin xyz="0 0 0" rpy="0 0 0" />
-      <geometry>
-        <mesh filename="package://robot/meshes/collision/right_hip_link.STL" />
+        <mesh filename="package://k1_description/meshes/visual/right_hip_link.STL" />
+      </geometry>
+      <material name="">
+        <color rgba="0.250980392156863 0.250980392156863 0.250980392156863 1" />
+      </material>
+    </visual>
+    <collision>
+      <origin xyz="0 0 0" rpy="0 0 0" />
+      <geometry>
+        <mesh filename="package://k1_description/meshes/collision/right_hip_link.STL" />
       </geometry>
     </collision>
@@ -59,14 +59,14 @@
       <origin xyz="0 0 0" rpy="0 0 0" />
       <geometry>
-        <mesh filename="package://robot/meshes/visual/right_thigh_link.STL" />
-      </geometry>
-      <material name="">
-        <color rgba="0.250980392156863 0.250980392156863 0.250980392156863 1" />
-      </material>
-    </visual>
-    <collision>
-      <origin xyz="0 0 0" rpy="0 0 0" />
-      <geometry>
-        <mesh filename="package://robot/meshes/collision/right_thigh_link.STL" />
+        <mesh filename="package://k1_description/meshes/visual/right_thigh_link.STL" />
+      </geometry>
+      <material name="">
+        <color rgba="0.250980392156863 0.250980392156863 0.250980392156863 1" />
+      </material>
+    </visual>
+    <collision>
+      <origin xyz="0 0 0" rpy="0 0 0" />
+      <geometry>
+        <mesh filename="package://k1_description/meshes/collision/right_thigh_link.STL" />
       </geometry>
     </collision>
@@ -87,14 +87,14 @@
       <origin xyz="0 0 0" rpy="0 0 0" />
       <geometry>
-        <mesh filename="package://robot/meshes/visual/right_knee_link.STL" />
-      </geometry>
-      <material name="">
-        <color rgba="0.752941176470588 1 1 1" />
-      </material>
-    </visual>
-    <collision>
-      <origin xyz="0 0 0" rpy="0 0 0" />
-      <geometry>
-        <mesh filename="package://robot/meshes/collision/right_knee_link.STL" />
+        <mesh filename="package://k1_description/meshes/visual/right_knee_link.STL" />
+      </geometry>
+      <material name="">
+        <color rgba="0.752941176470588 1 1 1" />
+      </material>
+    </visual>
+    <collision>
+      <origin xyz="0 0 0" rpy="0 0 0" />
+      <geometry>
+        <mesh filename="package://k1_description/meshes/collision/right_knee_link.STL" />
       </geometry>
     </collision>
@@ -115,14 +115,14 @@
       <origin xyz="0 0 0" rpy="0 0 0" />
       <geometry>
-        <mesh filename="package://robot/meshes/visual/right_calf_link.STL" />
-      </geometry>
-      <material name="">
-        <color rgba="0.752941176470588 1 1 1" />
-      </material>
-    </visual>
-    <collision>
-      <origin xyz="0 0 0" rpy="0 0 0" />
-      <geometry>
-        <mesh filename="package://robot/meshes/collision/right_calf_link.STL" />
+        <mesh filename="package://k1_description/meshes/visual/right_calf_link.STL" />
+      </geometry>
+      <material name="">
+        <color rgba="0.752941176470588 1 1 1" />
+      </material>
+    </visual>
+    <collision>
+      <origin xyz="0 0 0" rpy="0 0 0" />
+      <geometry>
+        <mesh filename="package://k1_description/meshes/collision/right_calf_link.STL" />
       </geometry>
     </collision>
@@ -143,14 +143,14 @@
       <origin xyz="0 0 0" rpy="0 0 0" />
       <geometry>
-        <mesh filename="package://robot/meshes/visual/right_ankle_link.STL" />
-      </geometry>
-      <material name="">
-        <color rgba="0.752941176470588 1 1 1" />
-      </material>
-    </visual>
-    <collision>
-      <origin xyz="0 0 0" rpy="0 0 0" />
-      <geometry>
-        <mesh filename="package://robot/meshes/collision/right_ankle_link.STL" />
+        <mesh filename="package://k1_description/meshes/visual/right_ankle_link.STL" />
+      </geometry>
+      <material name="">
+        <color rgba="0.752941176470588 1 1 1" />
+      </material>
+    </visual>
+    <collision>
+      <origin xyz="0 0 0" rpy="0 0 0" />
+      <geometry>
+        <mesh filename="package://k1_description/meshes/collision/right_ankle_link.STL" />
       </geometry>
     </collision>
@@ -171,14 +171,14 @@
       <origin xyz="0 0 0" rpy="0 0 0" />
       <geometry>
-        <mesh filename="package://robot/meshes/visual/left_hip_link.STL" />
-      </geometry>
-      <material name="">
-        <color rgba="0.250980392156863 0.250980392156863 0.250980392156863 1" />
-      </material>
-    </visual>
-    <collision>
-      <origin xyz="0 0 0" rpy="0 0 0" />
-      <geometry>
-        <mesh filename="package://robot/meshes/collision/left_hip_link.STL" />
+        <mesh filename="package://k1_description/meshes/visual/left_hip_link.STL" />
+      </geometry>
+      <material name="">
+        <color rgba="0.250980392156863 0.250980392156863 0.250980392156863 1" />
+      </material>
+    </visual>
+    <collision>
+      <origin xyz="0 0 0" rpy="0 0 0" />
+      <geometry>
+        <mesh filename="package://k1_description/meshes/collision/left_hip_link.STL" />
       </geometry>
     </collision>
@@ -199,14 +199,14 @@
       <origin xyz="0 0 0" rpy="0 0 0" />
       <geometry>
-        <mesh filename="package://robot/meshes/visual/left_thigh_link.STL" />
-      </geometry>
-      <material name="">
-        <color rgba="0.250980392156863 0.250980392156863 0.250980392156863 1" />
-      </material>
-    </visual>
-    <collision>
-      <origin xyz="0 0 0" rpy="0 0 0" />
-      <geometry>
-        <mesh filename="package://robot/meshes/collision/left_thigh_link.STL" />
+        <mesh filename="package://k1_description/meshes/visual/left_thigh_link.STL" />
+      </geometry>
+      <material name="">
+        <color rgba="0.250980392156863 0.250980392156863 0.250980392156863 1" />
+      </material>
+    </visual>
+    <collision>
+      <origin xyz="0 0 0" rpy="0 0 0" />
+      <geometry>
+        <mesh filename="package://k1_description/meshes/collision/left_thigh_link.STL" />
       </geometry>
     </collision>
@@ -227,14 +227,14 @@
       <origin xyz="0 0 0" rpy="0 0 0" />
       <geometry>
-        <mesh filename="package://robot/meshes/visual/left_knee_link.STL" />
-      </geometry>
-      <material name="">
-        <color rgba="0.752941176470588 1 1 1" />
-      </material>
-    </visual>
-    <collision>
-      <origin xyz="0 0 0" rpy="0 0 0" />
-      <geometry>
-        <mesh filename="package://robot/meshes/collision/left_knee_link.STL" />
+        <mesh filename="package://k1_description/meshes/visual/left_knee_link.STL" />
+      </geometry>
+      <material name="">
+        <color rgba="0.752941176470588 1 1 1" />
+      </material>
+    </visual>
+    <collision>
+      <origin xyz="0 0 0" rpy="0 0 0" />
+      <geometry>
+        <mesh filename="package://k1_description/meshes/collision/left_knee_link.STL" />
       </geometry>
     </collision>
@@ -255,14 +255,14 @@
       <origin xyz="0 0 0" rpy="0 0 0" />
       <geometry>
-        <mesh filename="package://robot/meshes/visual/left_calf_link.STL" />
-      </geometry>
-      <material name="">
-        <color rgba="0.752941176470588 1 1 1" />
-      </material>
-    </visual>
-    <collision>
-      <origin xyz="0 0 0" rpy="0 0 0" />
-      <geometry>
-        <mesh filename="package://robot/meshes/collision/left_calf_link.STL" />
+        <mesh filename="package://k1_description/meshes/visual/left_calf_link.STL" />
+      </geometry>
+      <material name="">
+        <color rgba="0.752941176470588 1 1 1" />
+      </material>
+    </visual>
+    <collision>
+      <origin xyz="0 0 0" rpy="0 0 0" />
+      <geometry>
+        <mesh filename="package://k1_description/meshes/collision/left_calf_link.STL" />
       </geometry>
     </collision>
@@ -283,14 +283,14 @@
       <origin xyz="0 0 0" rpy="0 0 0" />
       <geometry>
-        <mesh filename="package://robot/meshes/visual/left_ankle_link.STL" />
-      </geometry>
-      <material name="">
-        <color rgba="0.752941176470588 1 1 1" />
-      </material>
-    </visual>
-    <collision>
-      <origin xyz="0 0 0" rpy="0 0 0" />
-      <geometry>
-        <mesh filename="package://robot/meshes/collision/left_ankle_link.STL" />
+        <mesh filename="package://k1_description/meshes/visual/left_ankle_link.STL" />
+      </geometry>
+      <material name="">
+        <color rgba="0.752941176470588 1 1 1" />
+      </material>
+    </visual>
+    <collision>
+      <origin xyz="0 0 0" rpy="0 0 0" />
+      <geometry>
+        <mesh filename="package://k1_description/meshes/collision/left_ankle_link.STL" />
       </geometry>
     </collision>
@@ -311,14 +311,14 @@
       <origin xyz="0 0 0" rpy="0 0 0" />
       <geometry>
-        <mesh filename="package://robot/meshes/visual/right_shoulder_link.STL" />
-      </geometry>
-      <material name="">
-        <color rgba="0.752941176470588 1 1 1" />
-      </material>
-    </visual>
-    <collision>
-      <origin xyz="0 0 0" rpy="0 0 0" />
-      <geometry>
-        <mesh filename="package://robot/meshes/collision/right_shoulder_link.STL" />
+        <mesh filename="package://k1_description/meshes/visual/right_shoulder_link.STL" />
+      </geometry>
+      <material name="">
+        <color rgba="0.752941176470588 1 1 1" />
+      </material>
+    </visual>
+    <collision>
+      <origin xyz="0 0 0" rpy="0 0 0" />
+      <geometry>
+        <mesh filename="package://k1_description/meshes/collision/right_shoulder_link.STL" />
       </geometry>
     </collision>
@@ -339,14 +339,14 @@
       <origin xyz="0 0 0" rpy="0 0 0" />
       <geometry>
-        <mesh filename="package://robot/meshes/visual/right_upper_arm_link.STL" />
-      </geometry>
-      <material name="">
-        <color rgba="0.250980392156863 0.250980392156863 0.250980392156863 1" />
-      </material>
-    </visual>
-    <collision>
-      <origin xyz="0 0 0" rpy="0 0 0" />
-      <geometry>
-        <mesh filename="package://robot/meshes/collision/right_upper_arm_link.STL" />
+        <mesh filename="package://k1_description/meshes/visual/right_upper_arm_link.STL" />
+      </geometry>
+      <material name="">
+        <color rgba="0.250980392156863 0.250980392156863 0.250980392156863 1" />
+      </material>
+    </visual>
+    <collision>
+      <origin xyz="0 0 0" rpy="0 0 0" />
+      <geometry>
+        <mesh filename="package://k1_description/meshes/collision/right_upper_arm_link.STL" />
       </geometry>
     </collision>
@@ -367,14 +367,14 @@
       <origin xyz="0 0 0" rpy="0 0 0" />
       <geometry>
-        <mesh filename="package://robot/meshes/visual/right_lower_arm_link.STL" />
-      </geometry>
-      <material name="">
-        <color rgba="0.250980392156863 0.250980392156863 0.250980392156863 1" />
-      </material>
-    </visual>
-    <collision>
-      <origin xyz="0 0 0" rpy="0 0 0" />
-      <geometry>
-        <mesh filename="package://robot/meshes/collision/right_lower_arm_link.STL" />
+        <mesh filename="package://k1_description/meshes/visual/right_lower_arm_link.STL" />
+      </geometry>
+      <material name="">
+        <color rgba="0.250980392156863 0.250980392156863 0.250980392156863 1" />
+      </material>
+    </visual>
+    <collision>
+      <origin xyz="0 0 0" rpy="0 0 0" />
+      <geometry>
+        <mesh filename="package://k1_description/meshes/collision/right_lower_arm_link.STL" />
       </geometry>
     </collision>
@@ -395,14 +395,14 @@
       <origin xyz="0 0 0" rpy="0 0 0" />
       <geometry>
-        <mesh filename="package://robot/meshes/visual/left_shoulder_link.STL" />
-      </geometry>
-      <material name="">
-        <color rgba="0.752941176470588 1 1 1" />
-      </material>
-    </visual>
-    <collision>
-      <origin xyz="0 0 0" rpy="0 0 0" />
-      <geometry>
-        <mesh filename="package://robot/meshes/collision/left_shoulder_link.STL" />
+        <mesh filename="package://k1_description/meshes/visual/left_shoulder_link.STL" />
+      </geometry>
+      <material name="">
+        <color rgba="0.752941176470588 1 1 1" />
+      </material>
+    </visual>
+    <collision>
+      <origin xyz="0 0 0" rpy="0 0 0" />
+      <geometry>
+        <mesh filename="package://k1_description/meshes/collision/left_shoulder_link.STL" />
       </geometry>
     </collision>
@@ -423,14 +423,14 @@
       <origin xyz="0 0 0" rpy="0 0 0" />
       <geometry>
-        <mesh filename="package://robot/meshes/visual/left_upper_arm_link.STL" />
-      </geometry>
-      <material name="">
-        <color rgba="0.250980392156863 0.250980392156863 0.250980392156863 1" />
-      </material>
-    </visual>
-    <collision>
-      <origin xyz="0 0 0" rpy="0 0 0" />
-      <geometry>
-        <mesh filename="package://robot/meshes/collision/left_upper_arm_link.STL" />
+        <mesh filename="package://k1_description/meshes/visual/left_upper_arm_link.STL" />
+      </geometry>
+      <material name="">
+        <color rgba="0.250980392156863 0.250980392156863 0.250980392156863 1" />
+      </material>
+    </visual>
+    <collision>
+      <origin xyz="0 0 0" rpy="0 0 0" />
+      <geometry>
+        <mesh filename="package://k1_description/meshes/collision/left_upper_arm_link.STL" />
       </geometry>
     </collision>
@@ -451,14 +451,14 @@
       <origin xyz="0 0 0" rpy="0 0 0" />
       <geometry>
-        <mesh filename="package://robot/meshes/visual/left_lower_arm_link.STL" />
-      </geometry>
-      <material name="">
-        <color rgba="0.250980392156863 0.250980392156863 0.250980392156863 1" />
-      </material>
-    </visual>
-    <collision>
-      <origin xyz="0 0 0" rpy="0 0 0" />
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
Commit message: Switch back to revolute joints Signed-off-by: Curt Meyers <cmeyers@boilerbots.com>

File: ros2/src/k1_description/urdf/k1.xacro (robot description, xacro)
@@ -44,9 +44,10 @@
     </collision>
   </link>
-  <joint name="right_hip_joint" type="continuous">
+  <joint name="right_hip_joint" type="revolute">
     <origin xyz="-0.015 -0.000499999999999993 -0.02" rpy="-3.14159265358979 0.0316484172966858 -3.14159265358979" />
     <parent link="base_link" />
     <child link="right_hip_link" />
     <axis xyz="0 1 0" />
+    <limit lower="-6.0" upper="6.0" effort="1000" velocity="3.0" />
   </joint>
   <link name="right_thigh_link">
@@ -72,9 +73,10 @@
     </collision>
   </link>
-  <joint name="right_thigh_joint" type="continuous">
+  <joint name="right_thigh_joint" type="revolute">
     <origin xyz="0.0105 -0.000499999999999989 0.033" rpy="0 0.0253512899928625 -1.5707963267949" />
     <parent link="right_hip_link" />
     <child link="right_thigh_link" />
     <axis xyz="0 1 0" />
+    <limit lower="-6.0" upper="6.0" effort="1000" velocity="3.0" />
   </joint>
   <link name="right_knee_link">
@@ -100,9 +102,10 @@
     </collision>
   </link>
-  <joint name="right_knee_joint" type="continuous">
+  <joint name="right_knee_joint" type="revolute">
     <origin xyz="-0.00355599647142655 0 0.055419370059348" rpy="-3.14159265358978 -1.54544503680202 3.14159265358978" />
     <parent link="right_thigh_link" />
     <child link="right_knee_link" />
     <axis xyz="0 1 0" />
+    <limit lower="-6.0" upper="6.0" effort="1000" velocity="3.0" />
   </joint>
   <link name="right_calf_link">
@@ -128,9 +131,10 @@
     </collision>
   </link>
-  <joint name="right_calf_joint" type="continuous">
+  <joint name="right_calf_joint" type="revolute">
     <origin xyz="0.0566505085564426 0 0.00460572071266819" rpy="0 0 0" />
     <parent link="right_knee_link" />
     <child link="right_calf_link" />
     <axis xyz="0 1 0" />
+    <limit lower="-6.0" upper="6.0" effort="1000" velocity="3.0" />
   </joint>
   <link name="right_ankle_link">
@@ -156,9 +160,10 @@
     </collision>
   </link>
-  <joint name="right_ankle_joint" type="continuous">
+  <joint name="right_ankle_joint" type="revolute">
     <origin xyz="0.0330125603748861 -0.0074999999999983 0.000413349119391304" rpy="1.52798571545966 -0.000544427216642011 1.55808767255617" />
     <parent link="right_calf_link" />
     <child link="right_ankle_link" />
     <axis xyz="0 1 0" />
+    <limit lower="-6.0" upper="6.0" effort="1000" velocity="3.0" />
   </joint>
   <link name="left_hip_link">
@@ -184,9 +189,10 @@
     </collision>
   </link>
-  <joint name="left_hip_joint" type="continuous">
+  <joint name="left_hip_joint" type="revolute">
     <origin xyz="0.015 -0.000500000000000029 -0.02" rpy="3.14159265358979 -0.0788882616806473 0" />
     <parent link="base_link" />
     <child link="left_hip_link" />
     <axis xyz="0 1 0" />
+    <limit lower="-6.0" upper="6.0" effort="1000" velocity="3.0" />
   </joint>
   <link name="left_thigh_link">
@@ -212,9 +218,10 @@
     </collision>
   </link>
-  <joint name="left_thigh_joint" type="continuous">
+  <joint name="left_thigh_joint" type="revolute">
     <origin xyz="0.00899999999999999 0.000499999999999904 0.0329999999999999" rpy="1.5707963267949 -1.5707963267949 0" />
     <parent link="left_hip_link" />
     <child link="left_thigh_link" />
     <axis xyz="0 1 0" />
+    <limit lower="-6.0" upper="6.0" effort="1000" velocity="3.0" />
   </joint>
   <link name="left_knee_link">
@@ -240,9 +247,10 @@
     </collision>
   </link>
-  <joint name="left_knee_joint" type="continuous">
+  <joint name="left_knee_joint" type="revolute">
     <origin xyz="0.0554917017754941 0 0.0021500517992317" rpy="0 -1.01236160973997 0" />
     <parent link="left_thigh_link" />
     <child link="left_knee_link" />
     <axis xyz="0 1 0" />
+    <limit lower="-6.0" upper="6.0" effort="1000" velocity="3.0" />
   </joint>
   <link name="left_calf_link">
@@ -268,9 +276,10 @@
     </collision>
   </link>
-  <joint name="left_calf_joint" type="continuous">
+  <joint name="left_calf_joint" type="revolute">
     <origin xyz="0.0262634559672917 0 -0.0504055915910211" rpy="0 -0.581500701027345 0" />
     <parent link="left_knee_link" />
     <child link="left_calf_link" />
     <axis xyz="0 1 0" />
+    <limit lower="-6.0" upper="6.0" effort="1000" velocity="3.0" />
   </joint>
   <link name="left_ankle_link">
@@ -296,9 +305,10 @@
     </collision>
   </link>
-  <joint name="left_ankle_joint" type="continuous">
+  <joint name="left_ankle_joint" type="revolute">
     <origin xyz="-0.000999999999999996 0.00750000000000001 -0.033" rpy="0 0.0595977859512234 1.5707963267949" />
     <parent link="left_calf_link" />
     <child link="left_ankle_link" />
     <axis xyz="0 1 0" />
+    <limit lower="-6.0" upper="6.0" effort="1000" velocity="3.0" />
   </joint>
   <link name="right_shoulder_link">
@@ -324,9 +334,10 @@
     </collision>
   </link>
-  <joint name="right_shoulder_joint" type="continuous">
+  <joint name="right_shoulder_joint" type="revolute">
     <origin xyz="-0.026 0.00700000000000001 0.075" rpy="-3.14159265358979 0 -1.5707963267949" />
     <parent link="base_link" />
     <child link="right_shoulder_link" />
     <axis xyz="0 1 0" />
+    <limit lower="-6.0" upper="6.0" effort="1000" velocity="3.0" />
   </joint>
   <link name="right_upper_arm_link">
@@ -352,9 +363,10 @@
     </collision>
   </link>
-  <joint name="right_upper_arm_joint" type="continuous">
+  <joint name="right_upper_arm_joint" type="revolute">
     <origin xyz="0 0.0349999999999999 0" rpy="-0.00274508024652193 0.0285971009019822 1.57071783596033" />
     <parent link="right_shoulder_link" />
     <child link="right_upper_arm_link" />
     <axis xyz="0 1 0" />
+    <limit lower="-6.0" upper="6.0" effort="1000" velocity="3.0" />
   </joint>
   <link name="right_lower_arm_link">
@@ -380,9 +392,10 @@
     </collision>
   </link>
-  <joint name="right_lower_arm_joint" type="continuous">
+  <joint name="right_lower_arm_joint" type="revolute">
     <origin xyz="0 0 0.0699999999999956" rpy="0 -1.52080805151912 -1.57079632679487" />
     <parent link="right_upper_arm_link" />
     <child link="right_lower_arm_link" />
     <axis xyz="0 1 0" />
+    <limit lower="-6.0" upper="6.0" effort="1000" velocity="3.0" />
   </joint>
   <link name="left_shoulder_link">
@@ -408,9 +421,10 @@
     </collision>
   </link>
-  <joint name="left_shoulder_joint" type="continuous">
+  <joint name="left_shoulder_joint" type="revolute">
     <origin xyz="0.026 0.00700000000000001 0.075" rpy="3.14159265358979 0 -1.5707963267949" />
     <parent link="base_link" />
     <child link="left_shoulder_link" />
     <axis xyz="0 1 0" />
+    <limit lower="-6.0" upper="6.0" effort="1000" velocity="3.0" />
   </joint>
   <link name="left_upper_arm_link">
@@ -436,9 +450,10 @@
     </collision>
   </link>
-  <joint name="left_upper_arm_joint" type="continuous">
+  <joint name="left_upper_arm_joint" type="revolute">
     <origin xyz="0 -0.0349999999999999 0" rpy="0.00274508024652193 0.0285971009019818 1.57087481762947" />
     <parent link="left_shoulder_link" />
     <child link="left_upper_arm_link" />
     <axis xyz="0 1 0" />
+    <limit lower="-6.0" upper="6.0" effort="1000" velocity="3.0" />
   </joint>
   <link name="left_lower_arm_link">
@@ -464,9 +479,10 @@
     </collision>
   </link>
-  <joint name="left_lower_arm_joint" type="continuous">
+  <joint name="left_lower_arm_joint" type="revolute">
     <origin xyz="0 0 -0.0699999999999956" rpy="0 1.52080805151912 -1.57079632679494" />
     <parent link="left_upper_arm_link" />
     <child link="left_lower_arm_link" />
     <axis xyz="0 1 0" />
+    <limit lower="-6.0" upper="6.0" effort="1000" velocity="3.0" />
   </joint>
   <link name="head_link">
@@ -492,9 +508,10 @@
     </collision>
   </link>
-  <joint name="head_joint" type="continuous">
+  <joint name="head_joint" type="revolute">
     <origin xyz="0 0.011 0.071" rpy="-1.5707963267949 0 1.5707963267949" />
     <parent link="base_link" />
     <child link="head_link" />
     <axis xyz="0 1 0" />
+    <limit lower="-6.0" upper="6.0" effort="1000" velocity="3.0" />
   </joint>
 </robot>
