Commit message: Put left arm down
Signed-off-by: Curt Meyers <cmeyers@boilerbots.com>

File: ros2/src/k1_description/urdf/k1.xacro (robot description, xacro)
@@ -422,5 +422,5 @@
   </link>
   <joint name="left_shoulder_joint" type="revolute">
-    <origin xyz="0.026 0.00700000000000001 0.075" rpy="3.14159265358979 0 -1.5707963267949" />
+    <origin xyz="0.026 0.00700000000000001 0.075" rpy="0 0 -1.5707963267949" />
     <parent link="base_link" />
     <child link="left_shoulder_link" />
